File: HW/hodnoceni_LED.sch (KiCad schematic (older format))
At the start: 80 parts

Commit message: change structure of LEDs, add switching power supply of LEDs in parts
Parts:
- removed C? (x40): 100n, Capacitor_SMD:C_0402_1005Metric, symbol Device:C
- removed D? (x40): WS2812B, LED_SMD:LED_WS2812B_PLCC4_5.0x5.0mm_P3.2mm, symbol LED:WS2812B
Connections:
- no-connect marks 0 -> 1
