File: HW/zapinani.sch (KiCad schematic (older format))
At the start: 0 parts

Commit message: change structure of LEDs, add switching power supply of LEDs in parts
Parts:
- added Q?: Q_PMOS_DGS, symbol Device:Q_PMOS_DGS
- added R?: 10k, Resistor_SMD:R_0402_1005Metric, symbol Device:R
Connections:
- new net: Q?.2 (G), R?.1
- new net GPIO: R?.2
- new net V_BAT: Q?.3 (S)
- new net V_BAT_SPINANE: Q?.1 (D)
Other:
- note added: "IN\n"
- note added: "OUT\n"
Changed lines of the file:
@@
 $Descr A4 11693 8268
 encoding utf-8
-Sheet 1 22
+Sheet 22 42
 Title ""
 Date ""
@@
 Comment4 ""
 $EndDescr
+$Comp
+L Device:Q_PMOS_DGS Q?
+U 1 1 5F746478
+P 5100 2750
+AR Path="/5F746478" Ref="Q?"  Part="1"
+AR Path="/5F7BA54B/5F746478" Ref="Q?"  Part="1"
+AR Path="/5F7BA54B/5F7BCB45/5F746478" Ref="Q?"  Part="1"
+AR Path="/5F7BA54B/5F7BCBA6/5F746478" Ref="Q?"  Part="1"
+AR Path="/5F7BA54B/5F7BCC0A/5F746478" Ref="Q?"  Part="1"
+AR Path="/5F7BA54B/5F7BCC69/5F746478" Ref="Q?"  Part="1"
+F 0 "Q?" V 5442 2750 50  0000 C CNN
+F 1 "Q_PMOS_DGS" V 5351 2750 50  0000 C CNN
+F 2 "" H 5300 2850 50  0001 C CNN
+F 3 "~" H 5100 2750 50  0001 C CNN
+	1    5100 2750
+	0    -1   -1   0
+$EndComp
+$Comp
+L Device:R R?
+U 1 1 5F74647E
+P 5100 3250
+AR Path="/5F74647E" Ref="R?"  Part="1"
+AR Path="/5F7BA54B/5F74647E" Ref="R?"  Part="1"
+AR Path="/5F7BA54B/5F7BCB45/5F74647E" Ref="R?"  Part="1"
+AR Path="/5F7BA54B/5F7BCBA6/5F74647E" Ref="R?"  Part="1"
+AR Path="/5F7BA54B/5F7BCC0A/5F74647E" Ref="R?"  Part="1"
+AR Path="/5F7BA54B/5F7BCC69/5F74647E" Ref="R?"  Part="1"
+F 0 "R?" H 5170 3296 50  0000 L CNN
+F 1 "10k" H 5170 3205 50  0000 L CNN
+F 2 "Resistor_SMD:R_0402_1005Metric" V 5030 3250 50  0001 C CNN
+F 3 "~" H 5100 3250 50  0001 C CNN
+	1    5100 3250
+	1    0    0    -1
+$EndComp
+Wire Wire Line
+	4650 2650 4900 2650
+Wire Wire Line
+	5300 2650 5600 2650
+Wire Wire Line
+	5100 2950 5100 3100
+Wire Wire Line
+	5100 3400 5100 3550
+Text Notes 4200 2600 0    50   ~ 0
+IN\n
+Text Notes 5650 2600 0    50   ~ 0
+OUT\n
+Text HLabel 4650 2650 0    50   Input ~ 0
+V_BAT_SPINANE
+Text HLabel 5100 3550 3    50   Input ~ 0
+GPIO
+Text HLabel 5600 2650 2    50   Input ~ 0
+V_BAT
 $EndSCHEMATC
