File: HW/zapinani.sch (KiCad schematic (older format))
At the start: 2 parts, among them Q3 Q_PMOS_DGS

Commit message: continuation routing
Changed lines of the file:
@@
 $Descr A4 11693 8268
 encoding utf-8
-Sheet 18 34
+Sheet 33 34
 Title ""
 Date ""
@@
 AR Path="/5F7BA54B/5F7BCC0A/5F746478" Ref="Q5"  Part="1"
 AR Path="/5F7BA54B/5F7BCC69/5F746478" Ref="Q6"  Part="1"
-F 0 "Q4" V 5442 2750 50  0000 C CNN
+F 0 "Q3" V 5442 2750 50  0000 C CNN
 F 1 "Q_PMOS_DGS" V 5351 2750 50  0000 C CNN
 F 2 "Package_TO_SOT_SMD:SOT-23" H 5300 2850 50  0001 C CNN
@@
 AR Path="/5F7BA54B/5F7BCC0A/5F74647E" Ref="R16"  Part="1"
 AR Path="/5F7BA54B/5F7BCC69/5F74647E" Ref="R17"  Part="1"
-F 0 "R15" H 5170 3296 50  0000 L CNN
+F 0 "R14" H 5170 3296 50  0000 L CNN
 F 1 "10k" H 5170 3205 50  0000 L CNN
 F 2 "Resistor_SMD:R_0402_1005Metric" V 5030 3250 50  0001 C CNN

Commit message: ready for first prototype
Parts:
- Q3: JLCPCB_CORRECTION (none) -> 0;0;180
Changed lines of the file:
@@
 F 3 "~" H 5100 2750 50  0001 C CNN
 F 4 "C15127" H 5100 2750 50  0001 C CNN "LCSC"
+F 5 "0;0;180" H 5100 2750 50  0001 C CNN "JLCPCB_CORRECTION"
 	1    5100 2750
 	0    1    -1   0
