File: HW/Stepdown_ESP.sch (KiCad schematic (older format))
At the start: 12 parts

Commit message: add some packages
Parts:
- C? (x5): footprint (none) -> Capacitor_SMD:C_1206_3216Metric
- C?: footprint (none) -> Capacitor_SMD:C_0402_1005Metric
- L?: footprint (none) -> Inductor_SMD:L_0603_1608Metric
Other:
- note removed: "? co mám připojit na enable?\n"
Changed lines of the file:
@@
 $Descr A4 11693 8268
 encoding utf-8
-Sheet 14 42
+Sheet 12 42
 Title ""
 Date ""
@@
 F 0 "C?" H 4215 3646 50  0000 L CNN
 F 1 "22u" H 4215 3555 50  0000 L CNN
-F 2 "" H 4138 3450 50  0001 C CNN
+F 2 "Capacitor_SMD:C_1206_3216Metric" H 4138 3450 50  0001 C CNN
 F 3 "~" H 4100 3600 50  0001 C CNN
 	1    4100 3600
@@
 F 0 "C?" H 4665 3646 50  0000 L CNN
 F 1 "22u" H 4665 3555 50  0000 L CNN
-F 2 "" H 4588 3450 50  0001 C CNN
+F 2 "Capacitor_SMD:C_1206_3216Metric" H 4588 3450 50  0001 C CNN
 F 3 "~" H 4550 3600 50  0001 C CNN
 	1    4550 3600
@@
 F 0 "C?" H 5115 3646 50  0000 L CNN
 F 1 "22u" H 5115 3555 50  0000 L CNN
-F 2 "" H 5038 3450 50  0001 C CNN
+F 2 "Capacitor_SMD:C_1206_3216Metric" H 5038 3450 50  0001 C CNN
 F 3 "~" H 5000 3600 50  0001 C CNN
 	1    5000 3600
@@
 F 0 "L?" V 7290 3300 50  0000 C CNN
 F 1 "4u7" V 7199 3300 50  0000 C CNN
-F 2 "" H 7100 3300 50  0001 C CNN
+F 2 "Inductor_SMD:L_0603_1608Metric" H 7100 3300 50  0001 C CNN
 F 3 "~" H 7100 3300 50  0001 C CNN
 	1    7100 3300
@@
 F 0 "C?" H 8085 3504 50  0000 R CNN
 F 1 "47p" H 8085 3595 50  0000 R CNN
-F 2 "" H 8238 3400 50  0001 C CNN
+F 2 "Capacitor_SMD:C_0402_1005Metric" H 8238 3400 50  0001 C CNN
 F 3 "~" H 8200 3550 50  0001 C CNN
 	1    8200 3550
@@
 F 0 "C?" H 8585 3504 50  0000 R CNN
 F 1 "22u" H 8585 3595 50  0000 R CNN
-F 2 "" H 8738 3400 50  0001 C CNN
+F 2 "Capacitor_SMD:C_1206_3216Metric" H 8738 3400 50  0001 C CNN
 F 3 "~" H 8700 3550 50  0001 C CNN
 	1    8700 3550
@@
 F 0 "C?" H 8935 3504 50  0000 R CNN
 F 1 "22u" H 8935 3595 50  0000 R CNN
-F 2 "" H 9088 3400 50  0001 C CNN
+F 2 "Capacitor_SMD:C_1206_3216Metric" H 9088 3400 50  0001 C CNN
 F 3 "~" H 9050 3550 50  0001 C CNN
 	1    9050 3550
@@
 	6000 3300 5750 3300
 Connection ~ 5750 3300
-Text Notes 5100 3950 0    50   ~ 0
-? co mám připojit na enable?\n
-Wire Wire Line
-	5750 3800 5550 3800
-Connection ~ 5750 3800
 $EndSCHEMATC

Commit message: add polyfuse for battery, remove resistor by SY8105, fix mistake by charger
Parts:
- removed R?: 1M, Resistor_SMD:R_0402_1005Metric, symbol Device:R
Connections:
- net V_BAT_SPINANE: now also U?.2 (EN)
Changed lines of the file:
@@
 	5000 3300 4550 3300
 Connection ~ 4550 3300
-$Comp
-L Device:R R?
-U 1 1 602BA124
-P 5750 3600
-F 0 "R?" H 5820 3646 50  0000 L CNN
-F 1 "1M" H 5820 3555 50  0000 L CNN
-F 2 "Resistor_SMD:R_0402_1005Metric" V 5680 3600 50  0001 C CNN
-F 3 "~" H 5750 3600 50  0001 C CNN
-	1    5750 3600
-	1    0    0    -1
-$EndComp
-Wire Wire Line
-	5750 3450 5750 3300
 Wire Wire Line
 	5750 3300 5000 3300
@@
 	6000 3800 5750 3800
 Wire Wire Line
-	5750 3800 5750 3750
-Wire Wire Line
 	6000 3300 5750 3300
 Connection ~ 5750 3300
+Wire Wire Line
+	5750 3300 5750 3800
 $EndSCHEMATC
