File: HW/Stepdown_ESP.sch (KiCad schematic (older format))
At the start: 11 parts, among them U3 SY8105

Commit message: start place components
Parts:
- renumbered C20 to C27, C21 to C28, C22 to C29, C23 to C30, R8 to R11, R9 to R12
Connections:
- net V_BAT_SPINANE renamed +5V
Changed lines of the file:
@@
 $Descr A4 11693 8268
 encoding utf-8
-Sheet 5 30
+Sheet 5 28
 Title ""
 Date ""
@@
 $EndComp
 $Comp
-L power:GND #PWR0133
+L power:GND #PWR043
 U 1 1 602B858C
 P 4100 3900
-F 0 "#PWR0133" H 4100 3650 50  0001 C CNN
+F 0 "#PWR043" H 4100 3650 50  0001 C CNN
 F 1 "GND" H 4105 3727 50  0000 C CNN
 F 2 "" H 4100 3900 50  0001 C CNN
@@
 $EndComp
 $Comp
-L power:GND #PWR0134
+L power:GND #PWR044
 U 1 1 602B8981
 P 4550 3900
-F 0 "#PWR0134" H 4550 3650 50  0001 C CNN
+F 0 "#PWR044" H 4550 3650 50  0001 C CNN
 F 1 "GND" H 4555 3727 50  0000 C CNN
 F 2 "" H 4550 3900 50  0001 C CNN
@@
 $EndComp
 $Comp
-L power:GND #PWR0135
+L power:GND #PWR045
 U 1 1 602B8C3F
 P 5000 3900
-F 0 "#PWR0135" H 5000 3650 50  0001 C CNN
+F 0 "#PWR045" H 5000 3650 50  0001 C CNN
 F 1 "GND" H 5005 3727 50  0000 C CNN
 F 2 "" H 5000 3900 50  0001 C CNN
@@
 Wire Wire Line
 	5000 3750 5000 3900
-Text HLabel 3700 3300 0    50   Input ~ 0
-V_BAT_SPINANE
 Wire Wire Line
 	4100 3450 4100 3300
@@
 Connection ~ 5000 3300
 $Comp
-L Device:R R8
+L Device:R R11
 U 1 1 602BA607
 P 7450 3500
-F 0 "R8" H 7520 3546 50  0000 L CNN
+F 0 "R11" H 7520 3546 50  0000 L CNN
 F 1 "160k" H 7520 3455 50  0000 L CNN
 F 2 "Resistor_SMD:R_0603_1608Metric" V 7380 3500 50  0001 C CNN
@@
 $EndComp
 $Comp
-L Device:R R9
+L Device:R R12
 U 1 1 602BAA94
 P 7450 4050
-F 0 "R9" H 7520 4096 50  0000 L CNN
+F 0 "R12" H 7520 4096 50  0000 L CNN
 F 1 "36k" H 7520 4005 50  0000 L CNN
 F 2 "Resistor_SMD:R_0603_1608Metric" V 7380 4050 50  0001 C CNN
@@
 $EndComp
 $Comp
-L power:GND #PWR0136
+L power:GND #PWR046
 U 1 1 602BACDD
 P 6350 4350
-F 0 "#PWR0136" H 6350 4100 50  0001 C CNN
+F 0 "#PWR046" H 6350 4100 50  0001 C CNN
 F 1 "GND" H 6355 4177 50  0000 C CNN
 F 2 "" H 6350 4350 50  0001 C CNN
@@
 	7450 3300 7450 3350
 $Comp
-L Device:C C20
+L Device:C C27
 U 1 1 602BBFE2
 P 6650 2900
-F 0 "C20" V 6398 2900 50  0000 C CNN
+F 0 "C27" V 6398 2900 50  0000 C CNN
 F 1 "100n" V 6489 2900 50  0000 C CNN
 F 2 "Capacitor_SMD:C_0402_1005Metric" H 6688 2750 50  0001 C CNN
@@
 	6850 2900 6800 2900
 $Comp
-L Device:C C21
+L Device:C C28
 U 1 1 602BC82B
 P 8200 3550
-F 0 "C21" H 8085 3504 50  0000 R CNN
+F 0 "C28" H 8085 3504 50  0000 R CNN
 F 1 "47p" H 8085 3595 50  0000 R CNN
 F 2 "Capacitor_SMD:C_0402_1005Metric" H 8238 3400 50  0001 C CNN
@@
 $EndComp
 $Comp
-L Device:C C22
+L Device:C C29
 U 1 1 602BCF23
 P 8700 3550
-F 0 "C22" H 8585 3504 50  0000 R CNN
+F 0 "C29" H 8585 3504 50  0000 R CNN
 F 1 "22u" H 8585 3595 50  0000 R CNN
 F 2 "Capacitor_SMD:C_0603_1608Metric" H 8738 3400 50  0001 C CNN
@@
 $EndComp
 $Comp
-L Device:C C23
+L Device:C C30
 U 1 1 602BD148
 P 9050 3550
-F 0 "C23" H 8935 3504 50  0000 R CNN
+F 0 "C30" H 8935 3504 50  0000 R CNN
 F 1 "22u" H 8935 3595 50  0000 R CNN
 F 2 "Capacitor_SMD:C_0603_1608Metric" H 9088 3400 50  0001 C CNN
@@
 	7450 3800 7450 3650
 $Comp
-L power:GND #PWR0137
+L power:GND #PWR047
 U 1 1 602BE5D8
 P 8700 3850
-F 0 "#PWR0137" H 8700 3600 50  0001 C CNN
+F 0 "#PWR047" H 8700 3600 50  0001 C CNN
 F 1 "GND" H 8705 3677 50  0000 C CNN
 F 2 "" H 8700 3850 50  0001 C CNN
@@
 $EndComp
 $Comp
-L power:GND #PWR0138
+L power:GND #PWR048
 U 1 1 602BE8AF
 P 9050 3850
-F 0 "#PWR0138" H 9050 3600 50  0001 C CNN
+F 0 "#PWR048" H 9050 3600 50  0001 C CNN
 F 1 "GND" H 9055 3677 50  0000 C CNN
 F 2 "" H 9050 3850 50  0001 C CNN
@@
 	9050 3700 9050 3850
 $Comp
-L power:+3V3 #PWR0139
+L power:+3V3 #PWR049
 U 1 1 602BF312
 P 9350 3300
-F 0 "#PWR0139" H 9350 3150 50  0001 C CNN
+F 0 "#PWR049" H 9350 3150 50  0001 C CNN
 F 1 "+3V3" V 9365 3428 50  0000 L CNN
 F 2 "" H 9350 3300 50  0001 C CNN
@@
 Wire Wire Line
 	5750 3300 5750 3800
+$Comp
+L power:+5V #PWR?
+U 1 1 5FBB0D1E
+P 3700 3300
+F 0 "#PWR?" H 3700 3150 50  0001 C CNN
+F 1 "+5V" V 3715 3428 50  0000 L CNN
+F 2 "" H 3700 3300 50  0001 C CNN
+F 3 "" H 3700 3300 50  0001 C CNN
+	1    3700 3300
+	0    -1   -1   0
+$EndComp
 $EndSCHEMATC

Commit message: repair footprint of P and N MOS, add order codes for JLCPCB, preparing for fab
Parts:
- C24, C25, C26, C27, C28, C29, C30, L1, R11, R12: JLCPCB_CORRECTION (none) -> 0;0;0
Changed lines of the file:
@@
 F 3 "~" H 4100 3600 50  0001 C CNN
 F 4 "C59461" H 4100 3600 50  0001 C CNN "LCSC"
+F 5 "0;0;0" H 4100 3600 50  0001 C CNN "JLCPCB_CORRECTION"
 	1    4100 3600
 	1    0    0    -1
@@
 F 3 "~" H 4550 3600 50  0001 C CNN
 F 4 "C59461" H 4550 3600 50  0001 C CNN "LCSC"
+F 5 "0;0;0" H 4550 3600 50  0001 C CNN "JLCPCB_CORRECTION"
 	1    4550 3600
 	1    0    0    -1
@@
 F 3 "~" H 5000 3600 50  0001 C CNN
 F 4 "C59461" H 5000 3600 50  0001 C CNN "LCSC"
+F 5 "0;0;0" H 5000 3600 50  0001 C CNN "JLCPCB_CORRECTION"
 	1    5000 3600
 	1    0    0    -1
@@
 F 3 "~" H 7450 3500 50  0001 C CNN
 F 4 "C22813" H 7450 3500 50  0001 C CNN "LCSC"
+F 5 "0;0;0" H 7450 3500 50  0001 C CNN "JLCPCB_CORRECTION"
 	1    7450 3500
 	1    0    0    -1
@@
 F 3 "~" H 7450 4050 50  0001 C CNN
 F 4 "C23147" H 7450 4050 50  0001 C CNN "LCSC"
+F 5 "0;0;0" H 7450 4050 50  0001 C CNN "JLCPCB_CORRECTION"
 	1    7450 4050
 	1    0    0    -1
@@
 F 3 "~" H 7100 3300 50  0001 C CNN
 F 4 "C408410" H 7100 3300 50  0001 C CNN "LCSC"
+F 5 "0;0;0" H 7100 3300 50  0001 C CNN "JLCPCB_CORRECTION"
 	1    7100 3300
 	0    -1   -1   0
@@
 F 3 "~" H 6650 2900 50  0001 C CNN
 F 4 "C1525" H 6650 2900 50  0001 C CNN "LCSC"
+F 5 "0;0;0" H 6650 2900 50  0001 C CNN "JLCPCB_CORRECTION"
 	1    6650 2900
 	0    1    1    0
@@
 F 3 "~" H 8200 3550 50  0001 C CNN
 F 4 "C1567" H 8200 3550 50  0001 C CNN "LCSC"
+F 5 "0;0;0" H 8200 3550 50  0001 C CNN "JLCPCB_CORRECTION"
 	1    8200 3550
 	-1   0    0    1
@@
 F 3 "~" H 8700 3550 50  0001 C CNN
 F 4 "C59461" H 8700 3550 50  0001 C CNN "LCSC"
+F 5 "0;0;0" H 8700 3550 50  0001 C CNN "JLCPCB_CORRECTION"
 	1    8700 3550
 	-1   0    0    1
@@
 F 3 "~" H 9050 3550 50  0001 C CNN
 F 4 "C59461" H 9050 3550 50  0001 C CNN "LCSC"
+F 5 "0;0;0" H 9050 3550 50  0001 C CNN "JLCPCB_CORRECTION"
 	1    9050 3550
 	-1   0    0    1
