File: HW/Logic_KiCad - kopie.kicad_pcb (KiCad board)
At the start: 2 copper layers, 152 parts, among them J1 USB_B_Micro, Q1 Q_NPN_BCE, Q2 Q_NPN_BCE, Q3 Q_PMOS_DGS, Q4 Q_PMOS_DGS, Q7 Q_PMOS_DGS, SW1 SW_SPDT, SW10 button, SW11 button, SW12 button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

Commit message: finishing routing, make fab
Parts:
- moved C15 66.6 mm to (189.0, 79.6)
- moved SW11 66.6 mm to (178.4, 92.7)
- moved SW2 66.6 mm to (202.7, 92.5)
- moved SW6 66.6 mm to (186.2, 78.0)
- moved C109 66.6 mm to (197.5, 54.6)
- moved C11 66.6 mm to (205.4, 94.1)
- moved C111 66.6 mm to (205.1, 54.6)
- moved C113 66.6 mm to (212.6, 54.6)
- moved C115 66.6 mm to (220.1, 54.6)
- moved C119 66.6 mm to (204.9, 63.0)
- moved C12 66.6 mm to (147.0, 67.5)
- moved C121 66.6 mm to (212.3, 63.0)
- moved C123 66.6 mm to (220.0, 63.0)
- moved C125 66.6 mm to (197.3, 71.4)
- moved C127 66.6 mm to (204.8, 71.3)
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Routing:
- net +3V3: track 107.5 -> 69.8 mm, vias 8 -> 4
- net GND: track 1030.6 -> 1027.7 mm, vias 31 -> 10
- net VBUS: track 120.6 -> 121.7 mm
- net BARVA_2: track 114.4 -> 115.3 mm
- net BARVA_5: track 105.2 -> 105.9 mm
- net BARVA_4: track 94.1 -> 94.6 mm
