File: HW/zadani_LED.sch (KiCad schematic (older format))
At the start: 8 parts

Commit message: change structure of LEDs, add switching power supply of LEDs in parts
Connections:
- no-connect marks 0 -> 1
Changed lines of the file:
@@
 $Descr A4 11693 8268
 encoding utf-8
-Sheet 4 22
+Sheet 4 42
 Title ""
 Date ""
@@
 Text HLabel 2250 1500 0    50   Input ~ 0
 DATA_zadani_LED
-Text HLabel 1700 1000 0    50   Input ~ 0
-V_BAT
-Wire Wire Line
-	1700 1000 1950 1000
-Text GLabel 1950 1000 2    50   Input ~ 0
-V_BAT
-Text GLabel 3000 1100 0    50   Input ~ 0
+Text HLabel 2750 1100 0    50   Input ~ 0
 V_BAT
 Wire Wire Line
@@
 	7000 1100 6250 1100
 Connection ~ 6250 1100
+Wire Wire Line
+	2750 1100 3000 1100
+Connection ~ 3000 1100
+NoConn ~ 7300 1500
 $EndSCHEMATC

Commit message: add some codes for JLCPCB, change package and schematic of CP2102
Parts:
- C? (x4): LCSC (none) -> C1525
Changed lines of the file:
@@
 F 2 "Capacitor_SMD:C_0402_1005Metric" H 3588 1150 50  0001 C CNN
 F 3 "~" H 3550 1300 50  0001 C CNN
+F 4 "C1525" H 3550 1300 50  0001 C CNN "LCSC"
 	1    3550 1300
 	1    0    0    -1
@@
 F 2 "Capacitor_SMD:C_0402_1005Metric" H 4888 1150 50  0001 C CNN
 F 3 "~" H 4850 1300 50  0001 C CNN
+F 4 "C1525" H 4850 1300 50  0001 C CNN "LCSC"
 	1    4850 1300
 	1    0    0    -1
@@
 F 2 "Capacitor_SMD:C_0402_1005Metric" H 6288 1150 50  0001 C CNN
 F 3 "~" H 6250 1300 50  0001 C CNN
+F 4 "C1525" H 6250 1300 50  0001 C CNN "LCSC"
 	1    6250 1300
 	1    0    0    -1
@@
 F 2 "Capacitor_SMD:C_0402_1005Metric" H 7588 1150 50  0001 C CNN
 F 3 "~" H 7550 1300 50  0001 C CNN
+F 4 "C1525" H 7550 1300 50  0001 C CNN "LCSC"
 	1    7550 1300
 	1    0    0    -1

Commit message: add some codes for JLCPCB
Parts:
- D? (x4): LCSC (none) -> C114587
Changed lines of the file:
@@
 F 2 "LED_SMD:LED_WS2812B_PLCC4_5.0x5.0mm_P3.2mm" H 3050 1200 50  0001 L TNN
 F 3 "https://cdn-shop.adafruit.com/datasheets/WS2812B.pdf" H 3100 1125 50  0001 L TNN
+F 4 "C114587" H 3000 1500 50  0001 C CNN "LCSC"
 	1    3000 1500
 	1    0    0    -1
@@
 F 2 "LED_SMD:LED_WS2812B_PLCC4_5.0x5.0mm_P3.2mm" H 4350 1200 50  0001 L TNN
 F 3 "https://cdn-shop.adafruit.com/datasheets/WS2812B.pdf" H 4400 1125 50  0001 L TNN
+F 4 "C114587" H 4300 1500 50  0001 C CNN "LCSC"
 	1    4300 1500
 	1    0    0    -1
@@
 F 2 "LED_SMD:LED_WS2812B_PLCC4_5.0x5.0mm_P3.2mm" H 5750 1200 50  0001 L TNN
 F 3 "https://cdn-shop.adafruit.com/datasheets/WS2812B.pdf" H 5800 1125 50  0001 L TNN
+F 4 "C114587" H 5700 1500 50  0001 C CNN "LCSC"
 	1    5700 1500
 	1    0    0    -1
@@
 F 2 "LED_SMD:LED_WS2812B_PLCC4_5.0x5.0mm_P3.2mm" H 7050 1200 50  0001 L TNN
 F 3 "https://cdn-shop.adafruit.com/datasheets/WS2812B.pdf" H 7100 1125 50  0001 L TNN
+F 4 "C114587" H 7000 1500 50  0001 C CNN "LCSC"
 	1    7000 1500
 	1    0    0    -1

Commit message: numbering components, place components on board
Parts:
- gave numbers to parts that had none: 8
Changed lines of the file:
@@
 AR Path="/5FB77606" Ref="D?"  Part="1"
 AR Path="/5F70D6B6/5FB77606" Ref="D?"  Part="1"
-AR Path="/5FB682DC/5FB77606" Ref="D?"  Part="1"
-F 0 "D?" H 3344 1546 50  0000 L CNN
+AR Path="/5FB682DC/5FB77606" Ref="D2"  Part="1"
+F 0 "D2" H 3344 1546 50  0000 L CNN
 F 1 "WS2812B" H 3344 1455 50  0000 L CNN
 F 2 "LED_SMD:LED_WS2812B_PLCC4_5.0x5.0mm_P3.2mm" H 3050 1200 50  0001 L TNN
@@
 AR Path="/5FB7760C" Ref="#PWR?"  Part="1"
 AR Path="/5F70D6B6/5FB7760C" Ref="#PWR?"  Part="1"
-AR Path="/5FB682DC/5FB7760C" Ref="#PWR?"  Part="1"
-F 0 "#PWR?" H 3000 1650 50  0001 C CNN
+AR Path="/5FB682DC/5FB7760C" Ref="#PWR0111"  Part="1"
+F 0 "#PWR0111" H 3000 1650 50  0001 C CNN
 F 1 "GND" H 3005 1727 50  0000 C CNN
 F 2 "" H 3000 1900 50  0001 C CNN
@@
 AR Path="/5FB77618" Ref="C?"  Part="1"
 AR Path="/5F70D6B6/5FB77618" Ref="C?"  Part="1"
-AR Path="/5FB682DC/5FB77618" Ref="C?"  Part="1"
-F 0 "C?" H 3665 1346 50  0000 L CNN
+AR Path="/5FB682DC/5FB77618" Ref="C7"  Part="1"
+F 0 "C7" H 3665 1346 50  0000 L CNN
 F 1 "100n" H 3665 1255 50  0000 L CNN
 F 2 "Capacitor_SMD:C_0402_1005Metric" H 3588 1150 50  0001 C CNN
@@
 AR Path="/5FB77626" Ref="D?"  Part="1"
 AR Path="/5F70D6B6/5FB77626" Ref="D?"  Part="1"
-AR Path="/5FB682DC/5FB77626" Ref="D?"  Part="1"
-F 0 "D?" H 4644 1546 50  0000 L CNN
+AR Path="/5FB682DC/5FB77626" Ref="D3"  Part="1"
+F 0 "D3" H 4644 1546 50  0000 L CNN
 F 1 "WS2812B" H 4644 1455 50  0000 L CNN
 F 2 "LED_SMD:LED_WS2812B_PLCC4_5.0x5.0mm_P3.2mm" H 4350 1200 50  0001 L TNN
@@
 AR Path="/5FB7762C" Ref="#PWR?"  Part="1"
 AR Path="/5F70D6B6/5FB7762C" Ref="#PWR?"  Part="1"
-AR Path="/5FB682DC/5FB7762C" Ref="#PWR?"  Part="1"
-F 0 "#PWR?" H 4300 1650 50  0001 C CNN
+AR Path="/5FB682DC/5FB7762C" Ref="#PWR0112"  Part="1"
+F 0 "#PWR0112" H 4300 1650 50  0001 C CNN
 F 1 "GND" H 4305 1727 50  0000 C CNN
 F 2 "" H 4300 1900 50  0001 C CNN
@@
 AR Path="/5FB77638" Ref="C?"  Part="1"
 AR Path="/5F70D6B6/5FB77638" Ref="C?"  Part="1"
-AR Path="/5FB682DC/5FB77638" Ref="C?"  Part="1"
-F 0 "C?" H 4965 1346 50  0000 L CNN
+AR Path="/5FB682DC/5FB77638" Ref="C8"  Part="1"
+F 0 "C8" H 4965 1346 50  0000 L CNN
 F 1 "100n" H 4965 1255 50  0000 L CNN
 F 2 "Capacitor_SMD:C_0402_1005Metric" H 4888 1150 50  0001 C CNN
@@
 AR Path="/5FB77646" Ref="D?"  Part="1"
 AR Path="/5F70D6B6/5FB77646" Ref="D?"  Part="1"
-AR Path="/5FB682DC/5FB77646" Ref="D?"  Part="1"
-F 0 "D?" H 6044 1546 50  0000 L CNN
+AR Path="/5FB682DC/5FB77646" Ref="D4"  Part="1"
+F 0 "D4" H 6044 1546 50  0000 L CNN
 F 1 "WS2812B" H 6044 1455 50  0000 L CNN
 F 2 "LED_SMD:LED_WS2812B_PLCC4_5.0x5.0mm_P3.2mm" H 5750 1200 50  0001 L TNN
@@
 AR Path="/5FB7764C" Ref="#PWR?"  Part="1"
 AR Path="/5F70D6B6/5FB7764C" Ref="#PWR?"  Part="1"
-AR Path="/5FB682DC/5FB7764C" Ref="#PWR?"  Part="1"
-F 0 "#PWR?" H 5700 1650 50  0001 C CNN
+AR Path="/5FB682DC/5FB7764C" Ref="#PWR0113"  Part="1"
+F 0 "#PWR0113" H 5700 1650 50  0001 C CNN
 F 1 "GND" H 5705 1727 50  0000 C CNN
 F 2 "" H 5700 1900 50  0001 C CNN
@@
 AR Path="/5FB77658" Ref="C?"  Part="1"
 AR Path="/5F70D6B6/5FB77658" Ref="C?"  Part="1"
-AR Path="/5FB682DC/5FB77658" Ref="C?"  Part="1"
-F 0 "C?" H 6365 1346 50  0000 L CNN
+AR Path="/5FB682DC/5FB77658" Ref="C9"  Part="1"
+F 0 "C9" H 6365 1346 50  0000 L CNN
 F 1 "100n" H 6365 1255 50  0000 L CNN
 F 2 "Capacitor_SMD:C_0402_1005Metric" H 6288 1150 50  0001 C CNN
@@
 AR Path="/5FB77666" Ref="D?"  Part="1"
 AR Path="/5F70D6B6/5FB77666" Ref="D?"  Part="1"
-AR Path="/5FB682DC/5FB77666" Ref="D?"  Part="1"
-F 0 "D?" H 7344 1546 50  0000 L CNN
+AR Path="/5FB682DC/5FB77666" Ref="D5"  Part="1"
+F 0 "D5" H 7344 1546 50  0000 L CNN
 F 1 "WS2812B" H 7344 1455 50  0000 L CNN
 F 2 "LED_SMD:LED_WS2812B_PLCC4_5.0x5.0mm_P3.2mm" H 7050 1200 50  0001 L TNN
@@
 AR Path="/5FB7766C" Ref="#PWR?"  Part="1"
 AR Path="/5F70D6B6/5FB7766C" Ref="#PWR?"  Part="1"
-AR Path="/5FB682DC/5FB7766C" Ref="#PWR?"  Part="1"
-F 0 "#PWR?" H 7000 1650 50  0001 C CNN
+AR Path="/5FB682DC/5FB7766C" Ref="#PWR0114"  Part="1"
+F 0 "#PWR0114" H 7000 1650 50  0001 C CNN
 F 1 "GND" H 7005 1727 50  0000 C CNN
 F 2 "" H 7000 1900 50  0001 C CNN
@@
 AR Path="/5FB77678" Ref="C?"  Part="1"
 AR Path="/5F70D6B6/5FB77678" Ref="C?"  Part="1"
-AR Path="/5FB682DC/5FB77678" Ref="C?"  Part="1"
-F 0 "C?" H 7665 1346 50  0000 L CNN
+AR Path="/5FB682DC/5FB77678" Ref="C10"  Part="1"
+F 0 "C10" H 7665 1346 50  0000 L CNN
 F 1 "100n" H 7665 1255 50  0000 L CNN
 F 2 "Capacitor_SMD:C_0402_1005Metric" H 7588 1150 50  0001 C CNN
