File: HW/zadani_LED.sch (KiCad schematic (older format))
At the start: 8 parts

Commit message: start place components
Parts:
- renumbered D2 to D3, D3 to D4, D4 to D5, D5 to D6
Connections:
- net V_BAT renamed V_LED_1
Changed lines of the file:
@@
 $Descr A4 11693 8268
 encoding utf-8
-Sheet 2 30
+Sheet 2 28
 Title ""
 Date ""
@@
 AR Path="/5FB77606" Ref="D?"  Part="1"
 AR Path="/5F70D6B6/5FB77606" Ref="D?"  Part="1"
-AR Path="/5FB682DC/5FB77606" Ref="D2"  Part="1"
-F 0 "D2" H 3344 1546 50  0000 L CNN
+AR Path="/5FB682DC/5FB77606" Ref="D3"  Part="1"
+F 0 "D3" H 3344 1546 50  0000 L CNN
 F 1 "WS2812B" H 3344 1455 50  0000 L CNN
 F 2 "LED_SMD:LED_WS2812B_PLCC4_5.0x5.0mm_P3.2mm" H 3050 1200 50  0001 L TNN
@@
 AR Path="/5FB7760C" Ref="#PWR?"  Part="1"
 AR Path="/5F70D6B6/5FB7760C" Ref="#PWR?"  Part="1"
-AR Path="/5FB682DC/5FB7760C" Ref="#PWR0111"  Part="1"
-F 0 "#PWR0111" H 3000 1650 50  0001 C CNN
+AR Path="/5FB682DC/5FB7760C" Ref="#PWR016"  Part="1"
+F 0 "#PWR016" H 3000 1650 50  0001 C CNN
 F 1 "GND" H 3005 1727 50  0000 C CNN
 F 2 "" H 3000 1900 50  0001 C CNN
@@
 AR Path="/5FB77626" Ref="D?"  Part="1"
 AR Path="/5F70D6B6/5FB77626" Ref="D?"  Part="1"
-AR Path="/5FB682DC/5FB77626" Ref="D3"  Part="1"
-F 0 "D3" H 4644 1546 50  0000 L CNN
+AR Path="/5FB682DC/5FB77626" Ref="D4"  Part="1"
+F 0 "D4" H 4644 1546 50  0000 L CNN
 F 1 "WS2812B" H 4644 1455 50  0000 L CNN
 F 2 "LED_SMD:LED_WS2812B_PLCC4_5.0x5.0mm_P3.2mm" H 4350 1200 50  0001 L TNN
@@
 AR Path="/5FB7762C" Ref="#PWR?"  Part="1"
 AR Path="/5F70D6B6/5FB7762C" Ref="#PWR?"  Part="1"
-AR Path="/5FB682DC/5FB7762C" Ref="#PWR0112"  Part="1"
-F 0 "#PWR0112" H 4300 1650 50  0001 C CNN
+AR Path="/5FB682DC/5FB7762C" Ref="#PWR017"  Part="1"
+F 0 "#PWR017" H 4300 1650 50  0001 C CNN
 F 1 "GND" H 4305 1727 50  0000 C CNN
 F 2 "" H 4300 1900 50  0001 C CNN
@@
 AR Path="/5FB77646" Ref="D?"  Part="1"
 AR Path="/5F70D6B6/5FB77646" Ref="D?"  Part="1"
-AR Path="/5FB682DC/5FB77646" Ref="D4"  Part="1"
-F 0 "D4" H 6044 1546 50  0000 L CNN
+AR Path="/5FB682DC/5FB77646" Ref="D5"  Part="1"
+F 0 "D5" H 6044 1546 50  0000 L CNN
 F 1 "WS2812B" H 6044 1455 50  0000 L CNN
 F 2 "LED_SMD:LED_WS2812B_PLCC4_5.0x5.0mm_P3.2mm" H 5750 1200 50  0001 L TNN
@@
 AR Path="/5FB7764C" Ref="#PWR?"  Part="1"
 AR Path="/5F70D6B6/5FB7764C" Ref="#PWR?"  Part="1"
-AR Path="/5FB682DC/5FB7764C" Ref="#PWR0113"  Part="1"
-F 0 "#PWR0113" H 5700 1650 50  0001 C CNN
+AR Path="/5FB682DC/5FB7764C" Ref="#PWR018"  Part="1"
+F 0 "#PWR018" H 5700 1650 50  0001 C CNN
 F 1 "GND" H 5705 1727 50  0000 C CNN
 F 2 "" H 5700 1900 50  0001 C CNN
@@
 AR Path="/5FB77666" Ref="D?"  Part="1"
 AR Path="/5F70D6B6/5FB77666" Ref="D?"  Part="1"
-AR Path="/5FB682DC/5FB77666" Ref="D5"  Part="1"
-F 0 "D5" H 7344 1546 50  0000 L CNN
+AR Path="/5FB682DC/5FB77666" Ref="D6"  Part="1"
+F 0 "D6" H 7344 1546 50  0000 L CNN
 F 1 "WS2812B" H 7344 1455 50  0000 L CNN
 F 2 "LED_SMD:LED_WS2812B_PLCC4_5.0x5.0mm_P3.2mm" H 7050 1200 50  0001 L TNN
@@
 AR Path="/5FB7766C" Ref="#PWR?"  Part="1"
 AR Path="/5F70D6B6/5FB7766C" Ref="#PWR?"  Part="1"
-AR Path="/5FB682DC/5FB7766C" Ref="#PWR0114"  Part="1"
-F 0 "#PWR0114" H 7000 1650 50  0001 C CNN
+AR Path="/5FB682DC/5FB7766C" Ref="#PWR019"  Part="1"
+F 0 "#PWR019" H 7000 1650 50  0001 C CNN
 F 1 "GND" H 7005 1727 50  0000 C CNN
 F 2 "" H 7000 1900 50  0001 C CNN
@@
 DATA_zadani_LED
 Text HLabel 2750 1100 0    50   Input ~ 0
-V_BAT
+V_LED_1
 Wire Wire Line
 	4300 1100 3550 1100

Commit message: repair footprint of P and N MOS, add order codes for JLCPCB, preparing for fab
Parts:
- C10, C7, C8, C9: JLCPCB_CORRECTION (none) -> 0;0;0
- D3, D4, D5, D6: JLCPCB_CORRECTION (none) -> 0;0;90
Changed lines of the file:
@@
 F 3 "https://cdn-shop.adafruit.com/datasheets/WS2812B.pdf" H 3100 1125 50  0001 L TNN
 F 4 "C114587" H 3000 1500 50  0001 C CNN "LCSC"
+F 5 "0;0;90" H 3000 1500 50  0001 C CNN "JLCPCB_CORRECTION"
 	1    3000 1500
 	1    0    0    -1
@@
 F 3 "~" H 3550 1300 50  0001 C CNN
 F 4 "C1525" H 3550 1300 50  0001 C CNN "LCSC"
+F 5 "0;0;0" H 3550 1300 50  0001 C CNN "JLCPCB_CORRECTION"
 	1    3550 1300
 	1    0    0    -1
@@
 F 3 "https://cdn-shop.adafruit.com/datasheets/WS2812B.pdf" H 4400 1125 50  0001 L TNN
 F 4 "C114587" H 4300 1500 50  0001 C CNN "LCSC"
+F 5 "0;0;90" H 4300 1500 50  0001 C CNN "JLCPCB_CORRECTION"
 	1    4300 1500
 	1    0    0    -1
@@
 F 3 "~" H 4850 1300 50  0001 C CNN
 F 4 "C1525" H 4850 1300 50  0001 C CNN "LCSC"
+F 5 "0;0;0" H 4850 1300 50  0001 C CNN "JLCPCB_CORRECTION"
 	1    4850 1300
 	1    0    0    -1
@@
 F 3 "https://cdn-shop.adafruit.com/datasheets/WS2812B.pdf" H 5800 1125 50  0001 L TNN
 F 4 "C114587" H 5700 1500 50  0001 C CNN "LCSC"
+F 5 "0;0;90" H 5700 1500 50  0001 C CNN "JLCPCB_CORRECTION"
 	1    5700 1500
 	1    0    0    -1
@@
 F 3 "~" H 6250 1300 50  0001 C CNN
 F 4 "C1525" H 6250 1300 50  0001 C CNN "LCSC"
+F 5 "0;0;0" H 6250 1300 50  0001 C CNN "JLCPCB_CORRECTION"
 	1    6250 1300
 	1    0    0    -1
@@
 F 3 "https://cdn-shop.adafruit.com/datasheets/WS2812B.pdf" H 7100 1125 50  0001 L TNN
 F 4 "C114587" H 7000 1500 50  0001 C CNN "LCSC"
+F 5 "0;0;90" H 7000 1500 50  0001 C CNN "JLCPCB_CORRECTION"
 	1    7000 1500
 	1    0    0    -1
@@
 F 3 "~" H 7550 1300 50  0001 C CNN
 F 4 "C1525" H 7550 1300 50  0001 C CNN "LCSC"
+F 5 "0;0;0" H 7550 1300 50  0001 C CNN "JLCPCB_CORRECTION"
 	1    7550 1300
 	1    0    0    -1
