File: HW/zadani_LED.sch (KiCad schematic (older format))
At the start: 8 parts

Commit message: repair WS2812B na WS2812C
Parts:
- D3, D4, D5, D6: value WS2812B -> WS2812C
Changed lines of the file:
@@
 AR Path="/5FB682DC/5FB77606" Ref="D3"  Part="1"
 F 0 "D3" H 4194 3846 50  0000 L CNN
-F 1 "WS2812B" H 4194 3755 50  0000 L CNN
+F 1 "WS2812C" H 4194 3755 50  0000 L CNN
 F 2 "LED_SMD:LED_WS2812B_PLCC4_5.0x5.0mm_P3.2mm" H 3900 3500 50  0001 L TNN
 F 3 "https://cdn-shop.adafruit.com/datasheets/WS2812B.pdf" H 3950 3425 50  0001 L TNN
@@
 AR Path="/5FB682DC/5FB77626" Ref="D4"  Part="1"
 F 0 "D4" H 5494 3846 50  0000 L CNN
-F 1 "WS2812B" H 5494 3755 50  0000 L CNN
+F 1 "WS2812C" H 5494 3755 50  0000 L CNN
 F 2 "LED_SMD:LED_WS2812B_PLCC4_5.0x5.0mm_P3.2mm" H 5200 3500 50  0001 L TNN
 F 3 "https://cdn-shop.adafruit.com/datasheets/WS2812B.pdf" H 5250 3425 50  0001 L TNN
@@
 AR Path="/5FB682DC/5FB77646" Ref="D5"  Part="1"
 F 0 "D5" H 6894 3846 50  0000 L CNN
-F 1 "WS2812B" H 6894 3755 50  0000 L CNN
+F 1 "WS2812C" H 6894 3755 50  0000 L CNN
 F 2 "LED_SMD:LED_WS2812B_PLCC4_5.0x5.0mm_P3.2mm" H 6600 3500 50  0001 L TNN
 F 3 "https://cdn-shop.adafruit.com/datasheets/WS2812B.pdf" H 6650 3425 50  0001 L TNN
@@
 AR Path="/5FB682DC/5FB77666" Ref="D6"  Part="1"
 F 0 "D6" H 8194 3846 50  0000 L CNN
-F 1 "WS2812B" H 8194 3755 50  0000 L CNN
+F 1 "WS2812C" H 8194 3755 50  0000 L CNN
 F 2 "LED_SMD:LED_WS2812B_PLCC4_5.0x5.0mm_P3.2mm" H 7900 3500 50  0001 L TNN
 F 3 "https://cdn-shop.adafruit.com/datasheets/WS2812B.pdf" H 7950 3425 50  0001 L TNN

Commit message: update rotation of components for fab, update folder fab
Parts:
- D3, D4, D5, D6: JLCPCB_CORRECTION 0;0;90 -> 0;0;180
Changed lines of the file:
@@
 F 3 "https://cdn-shop.adafruit.com/datasheets/WS2812B.pdf" H 3950 3425 50  0001 L TNN
 F 4 "C114587" H 3850 3800 50  0001 C CNN "LCSC"
-F 5 "0;0;90" H 3850 3800 50  0001 C CNN "JLCPCB_CORRECTION"
+F 5 "0;0;180" H 3850 3800 50  0001 C CNN "JLCPCB_CORRECTION"
 	1    3850 3800
 	1    0    0    -1
@@
 F 3 "https://cdn-shop.adafruit.com/datasheets/WS2812B.pdf" H 5250 3425 50  0001 L TNN
 F 4 "C114587" H 5150 3800 50  0001 C CNN "LCSC"
-F 5 "0;0;90" H 5150 3800 50  0001 C CNN "JLCPCB_CORRECTION"
+F 5 "0;0;180" H 5150 3800 50  0001 C CNN "JLCPCB_CORRECTION"
 	1    5150 3800
 	1    0    0    -1
@@
 F 3 "https://cdn-shop.adafruit.com/datasheets/WS2812B.pdf" H 6650 3425 50  0001 L TNN
 F 4 "C114587" H 6550 3800 50  0001 C CNN "LCSC"
-F 5 "0;0;90" H 6550 3800 50  0001 C CNN "JLCPCB_CORRECTION"
+F 5 "0;0;180" H 6550 3800 50  0001 C CNN "JLCPCB_CORRECTION"
 	1    6550 3800
 	1    0    0    -1
@@
 F 3 "https://cdn-shop.adafruit.com/datasheets/WS2812B.pdf" H 7950 3425 50  0001 L TNN
 F 4 "C114587" H 7850 3800 50  0001 C CNN "LCSC"
-F 5 "0;0;90" H 7850 3800 50  0001 C CNN "JLCPCB_CORRECTION"
+F 5 "0;0;180" H 7850 3800 50  0001 C CNN "JLCPCB_CORRECTION"
 	1    7850 3800
 	1    0    0    -1
