File: HW/USB.sch (KiCad schematic (older format))
At the start: 4 parts, among them J1 USB_B_Micro

Commit message: update KiCad
Parts:
- J1: symbol Connector:USB_B_Micro -> Logic_KiCad-rescue:USB_B_Micro-Connector
Changed lines of the file:
@@
 $Descr A4 11693 8268
 encoding utf-8
-Sheet 19 21
+Sheet 8 21
 Title ""
 Date ""
@@
 $EndDescr
 $Comp
-L Connector:USB_B_Micro J?
+L Logic_KiCad-rescue:USB_B_Micro-Connector J?
 U 1 1 5F793175
 P 4000 3150

Commit message: deposit of DPS, start v1.0
Parts:
- removed D10, D11, D12: SD05_SOD323, Diode_SMD:D_SOD-323, symbol Diode:SD05_SOD323
- removed J1: USB_B_Micro, Connector_USB:USB_Micro-B_Wuerth_629105150521, symbol Logic_KiCad-rescue:USB_B_Micro-Connector
Connections:
- no-connect marks 1 -> 0
Changed lines of the file:
@@
 $Descr A4 11693 8268
 encoding utf-8
-Sheet 8 21
+Sheet 7 20
 Title ""
 Date ""
@@
 Comment4 ""
 $EndDescr
-$Comp
-L Logic_KiCad-rescue:USB_B_Micro-Connector J?
-U 1 1 5F793175
-P 4000 3150
-AR Path="/5F793175" Ref="J?"  Part="1"
-AR Path="/5FBB3550/5F793175" Ref="J?"  Part="1"
-AR Path="/5F78DB3E/5F793175" Ref="J1"  Part="1"
-F 0 "J1" H 4057 3617 50  0000 C CNN
-F 1 "USB_B_Micro" H 4057 3526 50  0000 C CNN
-F 2 "Connector_USB:USB_Micro-B_Wuerth_629105150521" H 4150 3100 50  0001 C CNN
-F 3 "~" H 4150 3100 50  0001 C CNN
-F 4 "ručně" H 4000 3150 50  0001 C CNN "LCSC"
-	1    4000 3150
-	1    0    0    -1
-$EndComp
-$Comp
-L power:GND #PWR?
-U 1 1 5F79317B
-P 4000 3550
-AR Path="/5FBB3550/5F79317B" Ref="#PWR?"  Part="1"
-AR Path="/5F79317B" Ref="#PWR?"  Part="1"
-AR Path="/5F78DB3E/5F79317B" Ref="#PWR0148"  Part="1"
-F 0 "#PWR0148" H 4000 3300 50  0001 C CNN
-F 1 "GND" H 4000 3400 50  0000 C CNN
-F 2 "" H 4000 3550 50  0001 C CNN
-F 3 "" H 4000 3550 50  0001 C CNN
-	1    4000 3550
-	1    0    0    -1
-$EndComp
-Wire Wire Line
-	4700 3150 4500 3150
-Wire Wire Line
-	4300 3250 4350 3250
-Wire Wire Line
-	4300 2950 4650 2950
-$Comp
-L Diode:SD05_SOD323 D?
-U 1 1 5F793184
-P 4350 3650
-AR Path="/5FBB3550/5F793184" Ref="D?"  Part="1"
-AR Path="/5F793184" Ref="D?"  Part="1"
-AR Path="/5F78DB3E/5F793184" Ref="D10"  Part="1"
-F 0 "D10" V 4400 3850 50  0000 R CNN
-F 1 "SD05_SOD323" V 4200 4200 50  0000 R CNN
-F 2 "Diode_SMD:D_SOD-323" H 4350 3450 50  0001 C CNN
-F 3 "https://www.littelfuse.com/~/media/electronics/datasheets/tvs_diode_arrays/littelfuse_tvs_diode_array_sd_c_datasheet.pdf.pdf" H 4350 3650 50  0001 C CNN
-F 4 "neosazovat" H 4350 3650 50  0001 C CNN "LCSC"
-	1    4350 3650
-	0    -1   -1   0
-$EndComp
-$Comp
-L Diode:SD05_SOD323 D?
-U 1 1 5F79318A
-P 4500 3650
-AR Path="/5FBB3550/5F79318A" Ref="D?"  Part="1"
-AR Path="/5F79318A" Ref="D?"  Part="1"
-AR Path="/5F78DB3E/5F79318A" Ref="D11"  Part="1"
-F 0 "D11" V 4650 3650 50  0000 R CNN
-F 1 "SD05_SOD323" V 4350 3650 50  0000 R CNN
-F 2 "Diode_SMD:D_SOD-323" H 4500 3450 50  0001 C CNN
-F 3 "https://www.littelfuse.com/~/media/electronics/datasheets/tvs_diode_arrays/littelfuse_tvs_diode_array_sd_c_datasheet.pdf.pdf" H 4500 3650 50  0001 C CNN
-F 4 "neosazovat" H 4500 3650 50  0001 C CNN "LCSC"
-	1    4500 3650
-	0    -1   -1   0
-$EndComp
-$Comp
-L Diode:SD05_SOD323 D?
-U 1 1 5F793190
-P 4650 3650
-AR Path="/5FBB3550/5F793190" Ref="D?"  Part="1"
-AR Path="/5F793190" Ref="D?"  Part="1"
-AR Path="/5F78DB3E/5F793190" Ref="D12"  Part="1"
-F 0 "D12" V 4696 3571 50  0000 R CNN
-F 1 "SD05_SOD323" V 4605 3571 50  0000 R CNN
-F 2 "Diode_SMD:D_SOD-323" H 4650 3450 50  0001 C CNN
-F 3 "https://www.littelfuse.com/~/media/electronics/datasheets/tvs_diode_arrays/littelfuse_tvs_diode_array_sd_c_datasheet.pdf.pdf" H 4650 3650 50  0001 C CNN
-F 4 "neosazovat" H 4650 3650 50  0001 C CNN "LCSC"
-	1    4650 3650
-	0    -1   -1   0
-$EndComp
-$Comp
-L power:GND #PWR?
-U 1 1 5F793196
-P 4350 3900
-AR Path="/5FBB3550/5F793196" Ref="#PWR?"  Part="1"
-AR Path="/5F793196" Ref="#PWR?"  Part="1"
-AR Path="/5F78DB3E/5F793196" Ref="#PWR0149"  Part="1"
-F 0 "#PWR0149" H 4350 3650 50  0001 C CNN
-F 1 "GND" H 4355 3727 50  0000 C CNN
-F 2 "" H 4350 3900 50  0001 C CNN
-F 3 "" H 4350 3900 50  0001 C CNN
-	1    4350 3900
-	1    0    0    -1
-$EndComp
-$Comp
-L power:GND #PWR?
-U 1 1 5F79319C
-P 4500 3900
-AR Path="/5FBB3550/5F79319C" Ref="#PWR?"  Part="1"
-AR Path="/5F79319C" Ref="#PWR?"  Part="1"
-AR Path="/5F78DB3E/5F79319C" Ref="#PWR0150"  Part="1"
-F 0 "#PWR0150" H 4500 3650 50  0001 C CNN
-F 1 "GND" H 4505 3727 50  0000 C CNN
-F 2 "" H 4500 3900 50  0001 C CNN
-F 3 "" H 4500 3900 50  0001 C CNN
-	1    4500 3900
-	1    0    0    -1
-$EndComp
-$Comp
-L power:GND #PWR?
-U 1 1 5F7931A2
-P 4650 3900
-AR Path="/5FBB3550/5F7931A2" Ref="#PWR?"  Part="1"
-AR Path="/5F7931A2" Ref="#PWR?"  Part="1"
-AR Path="/5F78DB3E/5F7931A2" Ref="#PWR0151"  Part="1"
-F 0 "#PWR0151" H 4650 3650 50  0001 C CNN
-F 1 "GND" H 4655 3727 50  0000 C CNN
-F 2 "" H 4650 3900 50  0001 C CNN
-F 3 "" H 4650 3900 50  0001 C CNN
-	1    4650 3900
-	1    0    0    -1
-$EndComp
-Wire Wire Line
-	4350 3800 4350 3900
-Wire Wire Line
-	4500 3800 4500 3900
-Wire Wire Line
-	4650 3800 4650 3900
-Wire Wire Line
-	4350 3500 4350 3250
-Connection ~ 4350 3250
-Wire Wire Line
-	4650 3500 4650 2950
-Connection ~ 4650 2950
-Wire Wire Line
-	4650 2950 4700 2950
-Wire Wire Line
-	4350 3250 4700 3250
-Wire Wire Line
-	4500 3500 4500 3150
-Connection ~ 4500 3150
-Wire Wire Line
-	4500 3150 4300 3150
-$Comp
-L power:GND #PWR?
-U 1 1 5F7931C2
-P 3900 3550
-AR Path="/5FBB3550/5F7931C2" Ref="#PWR?"  Part="1"
-AR Path="/5F7931C2" Ref="#PWR?"  Part="1"
-AR Path="/5F78DB3E/5F7931C2" Ref="#PWR0152"  Part="1"
-F 0 "#PWR0152" H 3900 3300 50  0001 C CNN
-F 1 "GND" H 3750 3500 50  0000 C CNN
-F 2 "" H 3900 3550 50  0001 C CNN
-F 3 "" H 3900 3550 50  0001 C CNN
-	1    3900 3550
-	1    0    0    -1
-$EndComp
-NoConn ~ 4300 3350
-Text HLabel 4700 3150 2    50   Input ~ 0
-D+
-Text HLabel 4700 3250 2    50   Input ~ 0
-D-
-Text HLabel 4700 2950 2    50   Input ~ 0
-VBUS
-$Comp
-L power:+5V #PWR?
-U 1 1 5F7931CC
-P 4650 2800
-AR Path="/5F7931CC" Ref="#PWR?"  Part="1"
-AR Path="/5F78DB3E/5F7931CC" Ref="#PWR0153"  Part="1"
-F 0 "#PWR0153" H 4650 2650 50  0001 C CNN
-F 1 "+5V" H 4665 2973 50  0000 C CNN
-F 2 "" H 4650 2800 50  0001 C CNN
-F 3 "" H 4650 2800 50  0001 C CNN
-	1    4650 2800
-	1    0    0    -1
-$EndComp
-Wire Wire Line
-	4650 2800 4650 2950
 $EndSCHEMATC
