File: HW/LEDky40.sch (KiCad schematic (older format))
At the start: 0 parts

Commit message: start place components
Changed lines of the file:
@@
 $Descr A4 11693 8268
 encoding utf-8
-Sheet 18 30
+Sheet 19 28
 Title ""
 Date ""
@@
 $EndDescr
 Text HLabel 1000 1000 0    50   Input ~ 0
-V_BAT_1
+V_LED_1
 Text HLabel 1000 800  0    50   Input ~ 0
 DATA_IN
@@
 $EndSheet
 Text HLabel 2650 1000 0    50   Input ~ 0
-V_BAT_1
+V_LED_1
 Wire Wire Line
 	2650 1000 2750 1000
@@
 $EndSheet
 Text HLabel 4150 1000 0    50   Input ~ 0
-V_BAT_1
+V_LED_1
 Wire Wire Line
 	4150 1000 4300 1000
@@
 F4 "V_BAT" I L 1250 1900 50
 $EndSheet
-Text HLabel 1000 1900 0    50   Input ~ 0
-V_BAT_2
 Wire Wire Line
 	1250 1700 1000 1700
@@
 NoConn ~ 2350 3600
 Text HLabel 2650 1900 0    50   Input ~ 0
-V_BAT_2
+V_LED_2
 Text HLabel 4150 1900 0    50   Input ~ 0
-V_BAT_2
+V_LED_2
 Wire Wire Line
 	4300 1900 4150 1900
 Wire Wire Line
 	2750 1900 2650 1900
-Text HLabel 1000 2800 0    50   Input ~ 0
-V_BAT_3
-Text HLabel 2650 2800 0    50   Input ~ 0
-V_BAT_3
+Text HLabel 4150 2800 0    50   Input ~ 0
+V_LED_3
 Wire Wire Line
 	2750 2800 2650 2800
 Wire Wire Line
 	1250 2800 1000 2800
-Text HLabel 4150 2800 0    50   Input ~ 0
-V_BAT_4
-Text HLabel 1000 3800 0    50   Input ~ 0
-V_BAT_4
 Wire Wire Line
 	4300 2800 4150 2800
 Wire Wire Line
 	1250 3800 1000 3800
+Text HLabel 1000 1900 0    50   Input ~ 0
+V_LED_1
+Text HLabel 2650 2800 0    50   Input ~ 0
+V_LED_3
+Text HLabel 1000 3800 0    50   Input ~ 0
+V_LED_3
+Text HLabel 1000 2800 0    50   Input ~ 0
+V_LED_2
 $EndSCHEMATC
