File: HW/Logic_KiCad_v0.kicad_pcb (KiCad board)
At the start: 2 copper layers, 92.5 x 82.5 mm, 152 parts, among them J1 USB_B_Micro, Q1 Q_NPN_BEC, Q2 Q_NPN_BEC, Q3 Q_PMOS_SDG, Q4 Q_PMOS_SDG, Q7 Q_PMOS_SDG, SW1 SW_SPDT, SW10 button, SW11 button, SW12 button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

Commit message: change footprint of buttons, continue placing components, repair mistake in power voltage
Other:
- board text added: "Logic v0 by Renata Zemanová"
- board text removed: "Logic v1.0 by Renata Zemanová"
