File: HW/LEDky4.sch (KiCad schematic (older format))
At the start: 8 parts

Commit message: start place components
Parts:
- renumbered C117 to C75, C119 to C76, C121 to C77, C123 to C78, D101 to D56, D103 to D57, D105 to D58, D107 to D59

Commit message: repair footprint of P and N MOS, add order codes for JLCPCB, preparing for fab
Parts:
- C75, C76, C77, C78: JLCPCB_CORRECTION (none) -> 0;0;0
- D56, D57, D58, D59: JLCPCB_CORRECTION (none) -> 0;0;90
Changed lines of the file:
@@
 $Descr A4 11693 8268
 encoding utf-8
-Sheet 29 28
+Sheet 10 28
 Title ""
 Date ""
@@
 AR Path="/5F79BCD0/5FB77CB0/5F78FD62" Ref="C67"  Part="1"
 AR Path="/5FACC290/5FB77CB0/5F78FD62" Ref="C107"  Part="1"
-F 0 "C107" H 2800 1650 50  0000 L CNN
+F 0 "C43" H 2800 1650 50  0000 L CNN
 F 1 "100n" H 2815 1555 50  0000 L CNN
 F 2 "Capacitor_SMD:C_0402_1005Metric" H 2738 1450 50  0001 C CNN
 F 3 "~" H 2700 1600 50  0001 C CNN
 F 4 "C1525" H 2700 1600 50  0001 C CNN "LCSC"
+F 5 "0;0;0" H 2700 1600 50  0001 C CNN "JLCPCB_CORRECTION"
 	1    2700 1600
 	1    0    0    -1
@@
 AR Path="/5F79BCD0/5FB77CB0/5F78FD71" Ref="D49"  Part="1"
 AR Path="/5FACC290/5FB77CB0/5F78FD71" Ref="D89"  Part="1"
-F 0 "D89" H 3894 1846 50  0000 L CNN
+F 0 "D25" H 3894 1846 50  0000 L CNN
 F 1 "WS2812B" H 3894 1755 50  0000 L CNN
 F 2 "LED_SMD:LED_WS2812B_PLCC4_5.0x5.0mm_P3.2mm" H 3600 1500 50  0001 L TNN
 F 3 "https://cdn-shop.adafruit.com/datasheets/WS2812B.pdf" H 3650 1425 50  0001 L TNN
 F 4 "C114587" H 3550 1800 50  0001 C CNN "LCSC"
+F 5 "0;0;90" H 3550 1800 50  0001 C CNN "JLCPCB_CORRECTION"
 	1    3550 1800
 	1    0    0    -1
@@
 AR Path="/5F79BCD0/5FB77CB0/5F78FDA5" Ref="D51"  Part="1"
 AR Path="/5FACC290/5FB77CB0/5F78FDA5" Ref="D91"  Part="1"
-F 0 "D91" H 6594 1846 50  0000 L CNN
+F 0 "D27" H 6594 1846 50  0000 L CNN
 F 1 "WS2812B" H 6594 1755 50  0000 L CNN
 F 2 "LED_SMD:LED_WS2812B_PLCC4_5.0x5.0mm_P3.2mm" H 6300 1500 50  0001 L TNN
 F 3 "https://cdn-shop.adafruit.com/datasheets/WS2812B.pdf" H 6350 1425 50  0001 L TNN
 F 4 "C114587" H 6250 1800 50  0001 C CNN "LCSC"
+F 5 "0;0;90" H 6250 1800 50  0001 C CNN "JLCPCB_CORRECTION"
 	1    6250 1800
 	1    0    0    -1
@@
 AR Path="/5F79BCD0/5FB77CB0/5F78FDB1" Ref="C70"  Part="1"
 AR Path="/5FACC290/5FB77CB0/5F78FDB1" Ref="C110"  Part="1"
-F 0 "C110" H 6915 1646 50  0000 L CNN
+F 0 "C46" H 6915 1646 50  0000 L CNN
 F 1 "100n" H 6915 1555 50  0000 L CNN
 F 2 "Capacitor_SMD:C_0402_1005Metric" H 6838 1450 50  0001 C CNN
 F 3 "~" H 6800 1600 50  0001 C CNN
 F 4 "C1525" H 6800 1600 50  0001 C CNN "LCSC"
+F 5 "0;0;0" H 6800 1600 50  0001 C CNN "JLCPCB_CORRECTION"
 	1    6800 1600
 	1    0    0    -1
@@
 AR Path="/5F79BCD0/5FB77CB0/5F78FD56" Ref="D48"  Part="1"
 AR Path="/5FACC290/5FB77CB0/5F78FD56" Ref="D88"  Part="1"
-F 0 "D88" H 2494 1846 50  0000 L CNN
+F 0 "D24" H 2494 1846 50  0000 L CNN
 F 1 "WS2812B" H 2494 1755 50  0000 L CNN
 F 2 "LED_SMD:LED_WS2812B_PLCC4_5.0x5.0mm_P3.2mm" H 2200 1500 50  0001 L TNN
 F 3 "https://cdn-shop.adafruit.com/datasheets/WS2812B.pdf" H 2250 1425 50  0001 L TNN
 F 4 "C114587" H 2150 1800 50  0001 C CNN "LCSC"
+F 5 "0;0;90" H 2150 1800 50  0001 C CNN "JLCPCB_CORRECTION"
 	1    2150 1800
 	1    0    0    -1
@@
 AR Path="/5F79BCD0/5FB77CB0/5F78FD7D" Ref="C68"  Part="1"
 AR Path="/5FACC290/5FB77CB0/5F78FD7D" Ref="C108"  Part="1"
-F 0 "C108" H 4215 1646 50  0000 L CNN
+F 0 "C44" H 4215 1646 50  0000 L CNN
 F 1 "100n" H 4215 1555 50  0000 L CNN
 F 2 "Capacitor_SMD:C_0402_1005Metric" H 4138 1450 50  0001 C CNN
 F 3 "~" H 4100 1600 50  0001 C CNN
 F 4 "C1525" H 4100 1600 50  0001 C CNN "LCSC"
+F 5 "0;0;0" H 4100 1600 50  0001 C CNN "JLCPCB_CORRECTION"
 	1    4100 1600
 	1    0    0    -1
@@
 AR Path="/5F79BCD0/5FB77CB0/5F78FD8B" Ref="D50"  Part="1"
 AR Path="/5FACC290/5FB77CB0/5F78FD8B" Ref="D90"  Part="1"
-F 0 "D90" H 5194 1846 50  0000 L CNN
+F 0 "D26" H 5194 1846 50  0000 L CNN
 F 1 "WS2812B" H 5194 1755 50  0000 L CNN
 F 2 "LED_SMD:LED_WS2812B_PLCC4_5.0x5.0mm_P3.2mm" H 4900 1500 50  0001 L TNN
 F 3 "https://cdn-shop.adafruit.com/datasheets/WS2812B.pdf" H 4950 1425 50  0001 L TNN
 F 4 "C114587" H 4850 1800 50  0001 C CNN "LCSC"
+F 5 "0;0;90" H 4850 1800 50  0001 C CNN "JLCPCB_CORRECTION"
 	1    4850 1800
 	1    0    0    -1
@@
 AR Path="/5F79BCD0/5FB77CB0/5F78FD97" Ref="C69"  Part="1"
 AR Path="/5FACC290/5FB77CB0/5F78FD97" Ref="C109"  Part="1"
-F 0 "C109" H 5515 1646 50  0000 L CNN
+F 0 "C45" H 5515 1646 50  0000 L CNN
 F 1 "100n" H 5515 1555 50  0000 L CNN
 F 2 "Capacitor_SMD:C_0402_1005Metric" H 5438 1450 50  0001 C CNN
 F 3 "~" H 5400 1600 50  0001 C CNN
 F 4 "C1525" H 5400 1600 50  0001 C CNN "LCSC"
+F 5 "0;0;0" H 5400 1600 50  0001 C CNN "JLCPCB_CORRECTION"
 	1    5400 1600
 	1    0    0    -1

Commit message: repair mistakes
Changed lines of the file:
@@
 AR Path="/5F79BCD0/5FB77CB0/5F78FD5C" Ref="#PWR0122"  Part="1"
 AR Path="/5FACC290/5FB77CB0/5F78FD5C" Ref="#PWR0207"  Part="1"
-F 0 "#PWR090" H 2150 1950 50  0001 C CNN
+F 0 "#PWR0207" H 2150 1950 50  0001 C CNN
 F 1 "GND" H 2155 2027 50  0000 C CNN
 F 2 "" H 2150 2200 50  0001 C CNN
@@
 AR Path="/5F79BCD0/5FB77CB0/5F78FD62" Ref="C67"  Part="1"
 AR Path="/5FACC290/5FB77CB0/5F78FD62" Ref="C107"  Part="1"
-F 0 "C43" H 2800 1650 50  0000 L CNN
+F 0 "C51" H 2800 1650 50  0000 L CNN
 F 1 "100n" H 2815 1555 50  0000 L CNN
 F 2 "Capacitor_SMD:C_0402_1005Metric" H 2738 1450 50  0001 C CNN
@@
 AR Path="/5F79BCD0/5FB77CB0/5F78FD71" Ref="D49"  Part="1"
 AR Path="/5FACC290/5FB77CB0/5F78FD71" Ref="D89"  Part="1"
-F 0 "D25" H 3894 1846 50  0000 L CNN
+F 0 "D33" H 3894 1846 50  0000 L CNN
 F 1 "WS2812B" H 3894 1755 50  0000 L CNN
 F 2 "LED_SMD:LED_WS2812B_PLCC4_5.0x5.0mm_P3.2mm" H 3600 1500 50  0001 L TNN
@@
 AR Path="/5F79BCD0/5FB77CB0/5F798BEB" Ref="#PWR0125"  Part="1"
 AR Path="/5FACC290/5FB77CB0/5F798BEB" Ref="#PWR0210"  Part="1"
-F 0 "#PWR093" H 3550 1950 50  0001 C CNN
+F 0 "#PWR0210" H 3550 1950 50  0001 C CNN
 F 1 "GND" H 3555 2027 50  0000 C CNN
 F 2 "" H 3550 2200 50  0001 C CNN
@@
 AR Path="/5F79BCD0/5FB77CB0/5F798BEE" Ref="#PWR0127"  Part="1"
 AR Path="/5FACC290/5FB77CB0/5F798BEE" Ref="#PWR0212"  Part="1"
-F 0 "#PWR095" H 4850 1950 50  0001 C CNN
+F 0 "#PWR0212" H 4850 1950 50  0001 C CNN
 F 1 "GND" H 4855 2027 50  0000 C CNN
 F 2 "" H 4850 2200 50  0001 C CNN
@@
 AR Path="/5F79BCD0/5FB77CB0/5F78FDA5" Ref="D51"  Part="1"
 AR Path="/5FACC290/5FB77CB0/5F78FDA5" Ref="D91"  Part="1"
-F 0 "D27" H 6594 1846 50  0000 L CNN
+F 0 "D35" H 6594 1846 50  0000 L CNN
 F 1 "WS2812B" H 6594 1755 50  0000 L CNN
 F 2 "LED_SMD:LED_WS2812B_PLCC4_5.0x5.0mm_P3.2mm" H 6300 1500 50  0001 L TNN
@@
 AR Path="/5F79BCD0/5FB77CB0/5F78FDAB" Ref="#PWR0128"  Part="1"
 AR Path="/5FACC290/5FB77CB0/5F78FDAB" Ref="#PWR0213"  Part="1"
-F 0 "#PWR096" H 6250 1950 50  0001 C CNN
+F 0 "#PWR0213" H 6250 1950 50  0001 C CNN
 F 1 "GND" H 6255 2027 50  0000 C CNN
 F 2 "" H 6250 2200 50  0001 C CNN
@@
 AR Path="/5F79BCD0/5FB77CB0/5F78FDB1" Ref="C70"  Part="1"
 AR Path="/5FACC290/5FB77CB0/5F78FDB1" Ref="C110"  Part="1"
-F 0 "C46" H 6915 1646 50  0000 L CNN
+F 0 "C54" H 6915 1646 50  0000 L CNN
 F 1 "100n" H 6915 1555 50  0000 L CNN
 F 2 "Capacitor_SMD:C_0402_1005Metric" H 6838 1450 50  0001 C CNN
@@
 AR Path="/5F79BCD0/5FB77CB0/5F78FD56" Ref="D48"  Part="1"
 AR Path="/5FACC290/5FB77CB0/5F78FD56" Ref="D88"  Part="1"
-F 0 "D24" H 2494 1846 50  0000 L CNN
+F 0 "D32" H 2494 1846 50  0000 L CNN
 F 1 "WS2812B" H 2494 1755 50  0000 L CNN
 F 2 "LED_SMD:LED_WS2812B_PLCC4_5.0x5.0mm_P3.2mm" H 2200 1500 50  0001 L TNN
@@
 AR Path="/5F79BCD0/5FB77CB0/5F798BE8" Ref="#PWR0123"  Part="1"
 AR Path="/5FACC290/5FB77CB0/5F798BE8" Ref="#PWR0208"  Part="1"
-F 0 "#PWR091" H 2150 1950 50  0001 C CNN
+F 0 "#PWR0208" H 2150 1950 50  0001 C CNN
 F 1 "GND" H 2155 2027 50  0000 C CNN
 F 2 "" H 2150 2200 50  0001 C CNN
@@
 AR Path="/5F79BCD0/5FB77CB0/5F78FD77" Ref="#PWR0124"  Part="1"
 AR Path="/5FACC290/5FB77CB0/5F78FD77" Ref="#PWR0209"  Part="1"
-F 0 "#PWR092" H 3550 1950 50  0001 C CNN
+F 0 "#PWR0209" H 3550 1950 50  0001 C CNN
 F 1 "GND" H 3555 2027 50  0000 C CNN
 F 2 "" H 3550 2200 50  0001 C CNN
@@
 AR Path="/5F79BCD0/5FB77CB0/5F78FD7D" Ref="C68"  Part="1"
 AR Path="/5FACC290/5FB77CB0/5F78FD7D" Ref="C108"  Part="1"
-F 0 "C44" H 4215 1646 50  0000 L CNN
+F 0 "C52" H 4215 1646 50  0000 L CNN
 F 1 "100n" H 4215 1555 50  0000 L CNN
 F 2 "Capacitor_SMD:C_0402_1005Metric" H 4138 1450 50  0001 C CNN
@@
 AR Path="/5F79BCD0/5FB77CB0/5F78FD8B" Ref="D50"  Part="1"
 AR Path="/5FACC290/5FB77CB0/5F78FD8B" Ref="D90"  Part="1"
-F 0 "D26" H 5194 1846 50  0000 L CNN
+F 0 "D34" H 5194 1846 50  0000 L CNN
 F 1 "WS2812B" H 5194 1755 50  0000 L CNN
 F 2 "LED_SMD:LED_WS2812B_PLCC4_5.0x5.0mm_P3.2mm" H 4900 1500 50  0001 L TNN
@@
 AR Path="/5F79BCD0/5FB77CB0/5F78FD91" Ref="#PWR0126"  Part="1"
 AR Path="/5FACC290/5FB77CB0/5F78FD91" Ref="#PWR0211"  Part="1"
-F 0 "#PWR094" H 4850 1950 50  0001 C CNN
+F 0 "#PWR0211" H 4850 1950 50  0001 C CNN
 F 1 "GND" H 4855 2027 50  0000 C CNN
 F 2 "" H 4850 2200 50  0001 C CNN
@@
 AR Path="/5F79BCD0/5FB77CB0/5F78FD97" Ref="C69"  Part="1"
 AR Path="/5FACC290/5FB77CB0/5F78FD97" Ref="C109"  Part="1"
-F 0 "C45" H 5515 1646 50  0000 L CNN
+F 0 "C53" H 5515 1646 50  0000 L CNN
 F 1 "100n" H 5515 1555 50  0000 L CNN
 F 2 "Capacitor_SMD:C_0402_1005Metric" H 5438 1450 50  0001 C CNN
@@
 AR Path="/5F79BCD0/5FB77CB0/5F798BF1" Ref="#PWR0129"  Part="1"
 AR Path="/5FACC290/5FB77CB0/5F798BF1" Ref="#PWR0214"  Part="1"
-F 0 "#PWR097" H 6250 1950 50  0001 C CNN
+F 0 "#PWR0214" H 6250 1950 50  0001 C CNN
 F 1 "GND" H 6255 2027 50  0000 C CNN
 F 2 "" H 6250 2200 50  0001 C CNN
