File: HW/zapinani_LEDek.sch (KiCad schematic (older format))
At the start: 12 parts, among them Q4 Q_NMOS_GSD, Q5 Q_PMOS_GSD, Q6 Q_NMOS_GSD, Q7 Q_PMOS_GSD, Q8 Q_NMOS_GSD, Q9 Q_PMOS_GSD

Commit message: repair mistakes
Parts:
- Q5, Q7, Q9: LCSC C8492 -> C15127
- R15, R17, R19: value 10k -> 100k; LCSC C25744 -> C25741
Changed lines of the file:
@@
 AR Path="/5F7BA54B/5F7BCC69/5F8EC656" Ref="R?"  Part="1"
 F 0 "R15" H 2420 3696 50  0000 L CNN
-F 1 "10k" H 2420 3605 50  0000 L CNN
+F 1 "100k" H 2420 3605 50  0000 L CNN
 F 2 "Resistor_SMD:R_0402_1005Metric" V 2280 3650 50  0001 C CNN
 F 3 "~" H 2350 3650 50  0001 C CNN
-F 4 "C25744" H 2350 3650 50  0001 C CNN "LCSC"
+F 4 "C25741" H 2350 3650 50  0001 C CNN "LCSC"
 F 5 "0;0;0" H 2350 3650 50  0001 C CNN "JLCPCB_CORRECTION"
 	1    2350 3650
@@
 AR Path="/5F7BA54B/5F7BCC69/5F8ECA6B" Ref="R?"  Part="1"
 F 0 "R17" H 5470 3646 50  0000 L CNN
-F 1 "10k" H 5470 3555 50  0000 L CNN
+F 1 "100k" H 5470 3555 50  0000 L CNN
 F 2 "Resistor_SMD:R_0402_1005Metric" V 5330 3600 50  0001 C CNN
 F 3 "~" H 5400 3600 50  0001 C CNN
-F 4 "C25744" H 5400 3600 50  0001 C CNN "LCSC"
+F 4 "C25741" H 5400 3600 50  0001 C CNN "LCSC"
 F 5 "0;0;0" H 5400 3600 50  0001 C CNN "JLCPCB_CORRECTION"
 	1    5400 3600
@@
 AR Path="/5F7BA54B/5F7BCC69/5FB8D0AF" Ref="R?"  Part="1"
 F 0 "R19" H 8320 3696 50  0000 L CNN
-F 1 "10k" H 8320 3605 50  0000 L CNN
+F 1 "100k" H 8320 3605 50  0000 L CNN
 F 2 "Resistor_SMD:R_0402_1005Metric" V 8180 3650 50  0001 C CNN
 F 3 "~" H 8250 3650 50  0001 C CNN
-F 4 "C25744" H 8250 3650 50  0001 C CNN "LCSC"
+F 4 "C25741" H 8250 3650 50  0001 C CNN "LCSC"
 F 5 "0;0;0" H 8250 3650 50  0001 C CNN "JLCPCB_CORRECTION"
 	1    8250 3650
@@
 F 2 "Package_TO_SOT_SMD:SOT-23" H 2850 3400 50  0001 C CNN
 F 3 "~" H 2650 3300 50  0001 C CNN
-F 4 "C8492" H 2650 3300 50  0001 C CNN "LCSC"
+F 4 "C15127" H 2650 3300 50  0001 C CNN "LCSC"
 F 5 "0;0;180" H 2650 3300 50  0001 C CNN "JLCPCB_CORRECTION"
 	1    2650 3300
@@
 F 2 "Package_TO_SOT_SMD:SOT-23" H 5900 3400 50  0001 C CNN
 F 3 "~" H 5700 3300 50  0001 C CNN
-F 4 "C8492" H 5700 3300 50  0001 C CNN "LCSC"
+F 4 "C15127" H 5700 3300 50  0001 C CNN "LCSC"
 F 5 "0;0;180" H 5700 3300 50  0001 C CNN "JLCPCB_CORRECTION"
 	1    5700 3300
@@
 F 2 "Package_TO_SOT_SMD:SOT-23" H 8750 3400 50  0001 C CNN
 F 3 "~" H 8550 3300 50  0001 C CNN
-F 4 "C8492" H 8550 3300 50  0001 C CNN "LCSC"
+F 4 "C15127" H 8550 3300 50  0001 C CNN "LCSC"
 F 5 "0;0;180" H 8550 3300 50  0001 C CNN "JLCPCB_CORRECTION"
 	1    8550 3300
