File: HW/USBto232.sch (KiCad schematic (older format))
At the start: 12 parts, among them Q1 Q_NPN_BCE, Q2 Q_NPN_BCE, U2 CP2102N-A01-GQFN28

Commit message: repair some misakes from prototype
Parts:
- removed Q1, Q2: Q_NPN_BCE, Package_TO_SOT_SMD:SOT-23, symbol Device:Q_NPN_BCE
- added Q1, Q2: Q_NPN_BEC, symbol Device:Q_NPN_BEC
Connections:
- wire segments 39 -> 45
Other:
- moved on the sheet: D7, R6

Commit message: deposit of DPS, start v1.0
Parts:
- added D? (x3): SD05_SOD323, Diode_SMD:D_SOD-323, symbol Diode:SD05_SOD323
- added J?: USB_B_Micro, Connector_USB:USB_Micro-B_Wuerth_629105150521, symbol Logic_KiCad-rescue:USB_B_Micro-Connector
Connections:
- net GND: now also D?.1 (A1), D?.1 (A1), D?.1 (A1), J?.5 (GND), J?.6 (Shield)
- net D+: no longer names the net of U2.4 (D+)
- net D+: now also D?.2 (A2), J?.3 (D+)
- net D-: no longer names the net of U2.5 (D-)
- net D-: now also D?.2 (A2), J?.2 (D-)
- net VBUS renamed +5V
- net +5V: now also D?.2 (A2), J?.1 (VBUS)
- no-connect marks 2 -> 3
Changed lines of the file:
@@
 $Descr A4 11693 8268
 encoding utf-8
-Sheet 4 21
+Sheet 4 30
 Title ""
 Date ""
@@
 Connection ~ 6150 1950
 Wire Wire Line
-	4650 3100 5000 3100
-Wire Wire Line
-	4650 3200 5000 3200
-Wire Wire Line
 	6650 3100 7050 3100
 Wire Wire Line
@@
 Wire Wire Line
 	6850 2100 6850 2200
-Text HLabel 4650 3000 0    50   Input ~ 0
-VBUS
-Text HLabel 4650 3100 0    50   Input ~ 0
-D+
-Text HLabel 4650 3200 0    50   Input ~ 0
-D-
 $Comp
 L Interface_USB:CP2102N-A01-GQFN28 U2
@@
 Wire Wire Line
 	6550 2500 6550 2800
+$Comp
+L power:+5V #PWR?
+U 1 1 5FB1FCC8
+P 4650 3000
+F 0 "#PWR?" H 4650 2850 50  0001 C CNN
+F 1 "+5V" V 4665 3128 50  0000 L CNN
+F 2 "" H 4650 3000 50  0001 C CNN
+F 3 "" H 4650 3000 50  0001 C CNN
+	1    4650 3000
+	0    -1   -1   0
+$EndComp
+$Comp
+L Logic_KiCad-rescue:USB_B_Micro-Connector J?
+U 1 1 5FB5E45C
+P 3300 3100
+AR Path="/5FB5E45C" Ref="J?"  Part="1"
+AR Path="/5FBB3550/5FB5E45C" Ref="J?"  Part="1"
+AR Path="/5F78DB3E/5FB5E45C" Ref="J?"  Part="1"
+F 0 "J?" H 3357 3567 50  0000 C CNN
+F 1 "USB_B_Micro" H 3357 3476 50  0000 C CNN
+F 2 "Connector_USB:USB_Micro-B_Wuerth_629105150521" H 3450 3050 50  0001 C CNN
+F 3 "~" H 3450 3050 50  0001 C CNN
+F 4 "ručně" H 3300 3100 50  0001 C CNN "LCSC"
+	1    3300 3100
+	1    0    0    -1
+$EndComp
+$Comp
+L power:GND #PWR?
+U 1 1 5FB5E462
+P 3300 3500
+AR Path="/5FBB3550/5FB5E462" Ref="#PWR?"  Part="1"
+AR Path="/5FB5E462" Ref="#PWR?"  Part="1"
+AR Path="/5F78DB3E/5FB5E462" Ref="#PWR?"  Part="1"
+F 0 "#PWR?" H 3300 3250 50  0001 C CNN
+F 1 "GND" H 3300 3350 50  0000 C CNN
+F 2 "" H 3300 3500 50  0001 C CNN
+F 3 "" H 3300 3500 50  0001 C CNN
+	1    3300 3500
+	1    0    0    -1
+$EndComp
+Wire Wire Line
+	3600 3200 3650 3200
+Wire Wire Line
+	3600 2900 3950 2900
+$Comp
+L Diode:SD05_SOD323 D?
+U 1 1 5FB5E46C
+P 3650 3600
+AR Path="/5FBB3550/5FB5E46C" Ref="D?"  Part="1"
+AR Path="/5FB5E46C" Ref="D?"  Part="1"
+AR Path="/5F78DB3E/5FB5E46C" Ref="D?"  Part="1"
+F 0 "D?" V 3700 3800 50  0000 R CNN
+F 1 "SD05_SOD323" V 3500 4150 50  0000 R CNN
+F 2 "Diode_SMD:D_SOD-323" H 3650 3400 50  0001 C CNN
+F 3 "https://www.littelfuse.com/~/media/electronics/datasheets/tvs_diode_arrays/littelfuse_tvs_diode_array_sd_c_datasheet.pdf.pdf" H 3650 3600 50  0001 C CNN
+F 4 "neosazovat" H 3650 3600 50  0001 C CNN "LCSC"
+	1    3650 3600
+	0    -1   -1   0
+$EndComp
+$Comp
+L Diode:SD05_SOD323 D?
+U 1 1 5FB5E473
+P 3800 3600
+AR Path="/5FBB3550/5FB5E473" Ref="D?"  Part="1"
+AR Path="/5FB5E473" Ref="D?"  Part="1"
+AR Path="/5F78DB3E/5FB5E473" Ref="D?"  Part="1"
+F 0 "D?" V 3950 3600 50  0000 R CNN
+F 1 "SD05_SOD323" V 3650 3600 50  0000 R CNN
+F 2 "Diode_SMD:D_SOD-323" H 3800 3400 50  0001 C CNN
+F 3 "https://www.littelfuse.com/~/media/electronics/datasheets/tvs_diode_arrays/littelfuse_tvs_diode_array_sd_c_datasheet.pdf.pdf" H 3800 3600 50  0001 C CNN
+F 4 "neosazovat" H 3800 3600 50  0001 C CNN "LCSC"
+	1    3800 3600
+	0    -1   -1   0
+$EndComp
+$Comp
+L Diode:SD05_SOD323 D?
+U 1 1 5FB5E47A
+P 3950 3600
+AR Path="/5FBB3550/5FB5E47A" Ref="D?"  Part="1"
+AR Path="/5FB5E47A" Ref="D?"  Part="1"
+AR Path="/5F78DB3E/5FB5E47A" Ref="D?"  Part="1"
+F 0 "D?" V 3996 3521 50  0000 R CNN
+F 1 "SD05_SOD323" V 3905 3521 50  0000 R CNN
+F 2 "Diode_SMD:D_SOD-323" H 3950 3400 50  0001 C CNN
+F 3 "https://www.littelfuse.com/~/media/electronics/datasheets/tvs_diode_arrays/littelfuse_tvs_diode_array_sd_c_datasheet.pdf.pdf" H 3950 3600 50  0001 C CNN
+F 4 "neosazovat" H 3950 3600 50  0001 C CNN "LCSC"
+	1    3950 3600
+	0    -1   -1   0
+$EndComp
+$Comp
+L power:GND #PWR?
+U 1 1 5FB5E480
+P 3650 3850
+AR Path="/5FBB3550/5FB5E480" Ref="#PWR?"  Part="1"
+AR Path="/5FB5E480" Ref="#PWR?"  Part="1"
+AR Path="/5F78DB3E/5FB5E480" Ref="#PWR?"  Part="1"
+F 0 "#PWR?" H 3650 3600 50  0001 C CNN
+F 1 "GND" H 3655 3677 50  0000 C CNN
+F 2 "" H 3650 3850 50  0001 C CNN
+F 3 "" H 3650 3850 50  0001 C CNN
+	1    3650 3850
+	1    0    0    -1
+$EndComp
+$Comp
+L power:GND #PWR?
+U 1 1 5FB5E486
+P 3800 3850
+AR Path="/5FBB3550/5FB5E486" Ref="#PWR?"  Part="1"
+AR Path="/5FB5E486" Ref="#PWR?"  Part="1"
+AR Path="/5F78DB3E/5FB5E486" Ref="#PWR?"  Part="1"
+F 0 "#PWR?" H 3800 3600 50  0001 C CNN
+F 1 "GND" H 3805 3677 50  0000 C CNN
+F 2 "" H 3800 3850 50  0001 C CNN
+F 3 "" H 3800 3850 50  0001 C CNN
+	1    3800 3850
+	1    0    0    -1
+$EndComp
+$Comp
+L power:GND #PWR?
+U 1 1 5FB5E48C
+P 3950 3850
+AR Path="/5FBB3550/5FB5E48C" Ref="#PWR?"  Part="1"
+AR Path="/5FB5E48C" Ref="#PWR?"  Part="1"
+AR Path="/5F78DB3E/5FB5E48C" Ref="#PWR?"  Part="1"
+F 0 "#PWR?" H 3950 3600 50  0001 C CNN
+F 1 "GND" H 3955 3677 50  0000 C CNN
+F 2 "" H 3950 3850 50  0001 C CNN
+F 3 "" H 3950 3850 50  0001 C CNN
+	1    3950 3850
+	1    0    0    -1
+$EndComp
+Wire Wire Line
+	3650 3750 3650 3850
+Wire Wire Line
+	3800 3750 3800 3850
+Wire Wire Line
+	3950 3750 3950 3850
+Wire Wire Line
+	3650 3450 3650 3200
+Connection ~ 3650 3200
+Wire Wire Line
+	3950 3450 3950 2900
+Connection ~ 3950 2900
+Wire Wire Line
+	3800 3450 3800 3100
+Connection ~ 3800 3100
+Wire Wire Line
+	3800 3100 3600 3100
+$Comp
+L power:GND #PWR?
+U 1 1 5FB5E49D
+P 3200 3500
+AR Path="/5FBB3550/5FB5E49D" Ref="#PWR?"  Part="1"
+AR Path="/5FB5E49D" Ref="#PWR?"  Part="1"
+AR Path="/5F78DB3E/5FB5E49D" Ref="#PWR?"  Part="1"
+F 0 "#PWR?" H 3200 3250 50  0001 C CNN
+F 1 "GND" H 3050 3450 50  0000 C CNN
+F 2 "" H 3200 3500 50  0001 C CNN
+F 3 "" H 3200 3500 50  0001 C CNN
+	1    3200 3500
+	1    0    0    -1
+$EndComp
+NoConn ~ 3600 3300
+$Comp
+L power:+5V #PWR?
+U 1 1 5FB5E4A6
+P 3950 2750
+AR Path="/5FB5E4A6" Ref="#PWR?"  Part="1"
+AR Path="/5F78DB3E/5FB5E4A6" Ref="#PWR?"  Part="1"
+AR Path="/5FBB3550/5FB5E4A6" Ref="#PWR?"  Part="1"
+F 0 "#PWR?" H 3950 2600 50  0001 C CNN
+F 1 "+5V" H 3965 2923 50  0000 C CNN
+F 2 "" H 3950 2750 50  0001 C CNN
+F 3 "" H 3950 2750 50  0001 C CNN
+	1    3950 2750
+	1    0    0    -1
+$EndComp
+Wire Wire Line
+	3950 2750 3950 2900
+Wire Wire Line
+	3800 3100 5000 3100
+Wire Wire Line
+	3650 3200 5000 3200
 $EndSCHEMATC

Commit message: start place components
Parts:
- Q1: renamed from Q2; footprint (none) -> Package_TO_SOT_SMD:SOT-23
- Q2: renamed from Q1; footprint (none) -> Package_TO_SOT_SMD:SOT-23
- gave numbers to parts that had none: 4
- renumbered C18 to C22, C19 to C23, D6 to D10, D7 to D11, R6 to R10, R5 to R6, R3 to R8, R4 to R9
Connections:
- net +5V: no longer D9.2 (A2), J1.1 (VBUS)
- new net V_OUT: D9.2 (A2), J1.1 (VBUS)
Changed lines of the file:
@@
 $Descr A4 11693 8268
 encoding utf-8
-Sheet 4 30
+Sheet 4 28
 Title ""
 Date ""
@@
 RX_ESP
 $Comp
-L power:GND #PWR0129
+L power:GND #PWR039
 U 1 1 5FBB9DA1
 P 5500 5000
-F 0 "#PWR0129" H 5500 4750 50  0001 C CNN
+F 0 "#PWR039" H 5500 4750 50  0001 C CNN
 F 1 "GND" H 5505 4827 50  0000 C CNN
 F 2 "" H 5500 5000 50  0001 C CNN
@@
 $EndComp
 $Comp
-L Device:R R5
+L Device:R R6
 U 1 1 5FBBF20B
 P 4500 2500
-F 0 "R5" H 4570 2546 50  0000 L CNN
+F 0 "R6" H 4570 2546 50  0000 L CNN
 F 1 "2k" H 4570 2455 50  0000 L CNN
 F 2 "Resistor_SMD:R_0402_1005Metric" V 4430 2500 50  0001 C CNN
@@
 EN_ESP
 $Comp
-L Device:R R6
+L Device:R R10
 U 1 1 5FBC5F56
 P 7550 2700
-F 0 "R6" V 7343 2700 50  0000 C CNN
+F 0 "R10" V 7343 2700 50  0000 C CNN
 F 1 "10k" V 7434 2700 50  0000 C CNN
 F 2 "Resistor_SMD:R_0402_1005Metric" V 7480 2700 50  0001 C CNN
@@
 	4500 2800 5000 2800
 $Comp
-L power:+3V3 #PWR0130
+L power:+3V3 #PWR036
 U 1 1 5FBD3E19
 P 4500 2300
-F 0 "#PWR0130" H 4500 2150 50  0001 C CNN
+F 0 "#PWR036" H 4500 2150 50  0001 C CNN
 F 1 "+3V3" H 4515 2473 50  0000 C CNN
 F 2 "" H 4500 2300 50  0001 C CNN
@@
 $EndComp
 $Comp
-L power:+3V3 #PWR0131
+L power:+3V3 #PWR038
 U 1 1 5FBD58C4
 P 5500 1900
-F 0 "#PWR0131" H 5500 1750 50  0001 C CNN
+F 0 "#PWR038" H 5500 1750 50  0001 C CNN
 F 1 "+3V3" H 5515 2073 50  0000 C CNN
 F 2 "" H 5500 1900 50  0001 C CNN
@@
 	5500 1900 5500 1950
 $Comp
-L Device:C C19
+L Device:C C23
 U 1 1 5FBD6F93
 P 5900 2250
-F 0 "C19" V 5950 2400 50  0000 C CNN
+F 0 "C23" V 5950 2400 50  0000 C CNN
 F 1 "100n" V 5750 2250 50  0000 C CNN
 F 2 "Capacitor_SMD:C_0402_1005Metric" H 5938 2100 50  0001 C CNN
@@
 	7350 3400 7600 3400
 $Comp
-L Device:R R3
+L Device:R R8
 U 1 1 5F7740AD
 P 6550 2350
-F 0 "R3" H 6620 2396 50  0000 L CNN
+F 0 "R8" H 6620 2396 50  0000 L CNN
 F 1 "47k" H 6620 2305 50  0000 L CNN
 F 2 "Resistor_SMD:R_0402_1005Metric" V 6480 2350 50  0001 C CNN
@@
 $EndComp
 $Comp
-L Device:R R4
+L Device:R R9
 U 1 1 5F774323
 P 6850 2350
-F 0 "R4" H 6920 2396 50  0000 L CNN
+F 0 "R9" H 6920 2396 50  0000 L CNN
 F 1 "47k" H 6920 2305 50  0000 L CNN
 F 2 "Resistor_SMD:R_0402_1005Metric" V 6780 2350 50  0001 C CNN
@@
 $EndComp
 $Comp
-L Device:LED D6
+L Device:LED D10
 U 1 1 5F774688
 P 6550 1950
-F 0 "D6" V 6550 2100 50  0000 R CNN
+F 0 "D10" V 6550 2150 50  0000 R CNN
 F 1 "green" V 6650 2200 50  0000 R CNN
 F 2 "LED_SMD:LED_0603_1608Metric" H 6550 1950 50  0001 C CNN
@@
 $EndComp
 $Comp
-L Device:LED D7
+L Device:LED D11
 U 1 1 5F774C1B
 P 6850 1950
-F 0 "D7" V 6800 2000 50  0000 L CNN
+F 0 "D11" V 6800 2000 50  0000 L CNN
 F 1 "green" V 6950 2000 50  0000 L CNN
 F 2 "LED_SMD:LED_0603_1608Metric" H 6850 1950 50  0001 C CNN
@@
 	4650 3000 5000 3000
 $Comp
-L Device:Q_NPN_BEC Q1
+L Device:Q_NPN_BEC Q2
 U 1 1 5FAEE7FB
 P 8050 2700
-F 0 "Q1" H 8241 2746 50  0000 L CNN
+F 0 "Q2" H 8241 2746 50  0000 L CNN
 F 1 "Q_NPN_BEC" H 8241 2655 50  0000 L CNN
-F 2 "" H 8250 2800 50  0001 C CNN
+F 2 "Package_TO_SOT_SMD:SOT-23" H 8250 2800 50  0001 C CNN
 F 3 "~" H 8050 2700 50  0001 C CNN
 	1    8050 2700
@@
 $EndComp
 $Comp
-L Device:Q_NPN_BEC Q2
+L Device:Q_NPN_BEC Q1
 U 1 1 5FAEE9BB
 P 7250 3100
-F 0 "Q2" H 7441 3054 50  0000 L CNN
+F 0 "Q1" H 7441 3054 50  0000 L CNN
 F 1 "Q_NPN_BEC" H 7441 3145 50  0000 L CNN
-F 2 "" H 7450 3200 50  0001 C CNN
+F 2 "Package_TO_SOT_SMD:SOT-23" H 7450 3200 50  0001 C CNN
 F 3 "~" H 7250 3100 50  0001 C CNN
 	1    7250 3100
@@
 $EndComp
 $Comp
-L power:+3V3 #PWR0126
+L power:+3V3 #PWR041
 U 1 1 5FAFF359
 P 6550 1650
-F 0 "#PWR0126" H 6550 1500 50  0001 C CNN
+F 0 "#PWR041" H 6550 1500 50  0001 C CNN
 F 1 "+3V3" H 6565 1823 50  0000 C CNN
 F 2 "" H 6550 1650 50  0001 C CNN
@@
 $EndComp
 $Comp
-L power:+3V3 #PWR0127
+L power:+3V3 #PWR042
 U 1 1 5FAFF4D0
 P 6850 1650
-F 0 "#PWR0127" H 6850 1500 50  0001 C CNN
+F 0 "#PWR042" H 6850 1500 50  0001 C CNN
 F 1 "+3V3" H 6865 1823 50  0000 C CNN
 F 2 "" H 6850 1650 50  0001 C CNN
@@
 	6050 1950 6150 1950
 $Comp
-L Device:C C18
+L Device:C C22
 U 1 1 5FBD67B7
 P 5900 1950
-F 0 "C18" V 5648 1950 50  0000 C CNN
+F 0 "C22" V 5648 1950 50  0000 C CNN
 F 1 "4u7" V 5739 1950 50  0000 C CNN
 F 2 "Capacitor_SMD:C_0402_1005Metric" H 5938 1800 50  0001 C CNN
@@
 	6200 1950 6150 1950
 $Comp
-L power:GND #PWR0132
+L power:GND #PWR040
 U 1 1 5FBD8F58
 P 6200 1950
-F 0 "#PWR0132" H 6200 1700 50  0001 C CNN
+F 0 "#PWR040" H 6200 1700 50  0001 C CNN
 F 1 "GND" V 6100 1950 50  0000 R CNN
 F 2 "" H 6200 1950 50  0001 C CNN
@@
 	6550 2500 6550 2800
 $Comp
-L power:+5V #PWR?
+L power:+5V #PWR037
 U 1 1 5FB1FCC8
 P 4650 3000
-F 0 "#PWR?" H 4650 2850 50  0001 C CNN
+F 0 "#PWR037" H 4650 2850 50  0001 C CNN
 F 1 "+5V" V 4665 3128 50  0000 L CNN
 F 2 "" H 4650 3000 50  0001 C CNN
@@
 P 3300 3100
 AR Path="/5FB5E45C" Ref="J?"  Part="1"
-AR Path="/5FBB3550/5FB5E45C" Ref="J?"  Part="1"
+AR Path="/5FBB3550/5FB5E45C" Ref="J1"  Part="1"
 AR Path="/5F78DB3E/5FB5E45C" Ref="J?"  Part="1"
-F 0 "J?" H 3357 3567 50  0000 C CNN
+F 0 "J1" H 3357 3567 50  0000 C CNN
 F 1 "USB_B_Micro" H 3357 3476 50  0000 C CNN
 F 2 "Connector_USB:USB_Micro-B_Wuerth_629105150521" H 3450 3050 50  0001 C CNN
@@
 $EndComp
 $Comp
-L power:GND #PWR?
+L power:GND #PWR032
 U 1 1 5FB5E462
 P 3300 3500
-AR Path="/5FBB3550/5FB5E462" Ref="#PWR?"  Part="1"
+AR Path="/5FBB3550/5FB5E462" Ref="#PWR032"  Part="1"
 AR Path="/5FB5E462" Ref="#PWR?"  Part="1"
 AR Path="/5F78DB3E/5FB5E462" Ref="#PWR?"  Part="1"
-F 0 "#PWR?" H 3300 3250 50  0001 C CNN
+F 0 "#PWR032" H 3300 3250 50  0001 C CNN
 F 1 "GND" H 3300 3350 50  0000 C CNN
 F 2 "" H 3300 3500 50  0001 C CNN
@@
 	3600 2900 3950 2900
 $Comp
-L Diode:SD05_SOD323 D?
+L Diode:SD05_SOD323 D7
 U 1 1 5FB5E46C
 P 3650 3600
-AR Path="/5FBB3550/5FB5E46C" Ref="D?"  Part="1"
+AR Path="/5FBB3550/5FB5E46C" Ref="D7"  Part="1"
 AR Path="/5FB5E46C" Ref="D?"  Part="1"
 AR Path="/5F78DB3E/5FB5E46C" Ref="D?"  Part="1"
-F 0 "D?" V 3700 3800 50  0000 R CNN
+F 0 "D7" V 3700 3800 50  0000 R CNN
 F 1 "SD05_SOD323" V 3500 4150 50  0000 R CNN
 F 2 "Diode_SMD:D_SOD-323" H 3650 3400 50  0001 C CNN
@@
 $EndComp
 $Comp
-L Diode:SD05_SOD323 D?
+L Diode:SD05_SOD323 D8
 U 1 1 5FB5E473
 P 3800 3600
-AR Path="/5FBB3550/5FB5E473" Ref="D?"  Part="1"
+AR Path="/5FBB3550/5FB5E473" Ref="D8"  Part="1"
 AR Path="/5FB5E473" Ref="D?"  Part="1"
 AR Path="/5F78DB3E/5FB5E473" Ref="D?"  Part="1"
-F 0 "D?" V 3950 3600 50  0000 R CNN
+F 0 "D8" V 3950 3600 50  0000 R CNN
 F 1 "SD05_SOD323" V 3650 3600 50  0000 R CNN
 F 2 "Diode_SMD:D_SOD-323" H 3800 3400 50  0001 C CNN
@@
 $EndComp
 $Comp
-L Diode:SD05_SOD323 D?
+L Diode:SD05_SOD323 D9
 U 1 1 5FB5E47A
 P 3950 3600
-AR Path="/5FBB3550/5FB5E47A" Ref="D?"  Part="1"
+AR Path="/5FBB3550/5FB5E47A" Ref="D9"  Part="1"
 AR Path="/5FB5E47A" Ref="D?"  Part="1"
 AR Path="/5F78DB3E/5FB5E47A" Ref="D?"  Part="1"
-F 0 "D?" V 3996 3521 50  0000 R CNN
+F 0 "D9" V 3996 3521 50  0000 R CNN
 F 1 "SD05_SOD323" V 3905 3521 50  0000 R CNN
 F 2 "Diode_SMD:D_SOD-323" H 3950 3400 50  0001 C CNN
@@
 $EndComp
 $Comp
-L power:GND #PWR?
+L power:GND #PWR033
 U 1 1 5FB5E480
 P 3650 3850
-AR Path="/5FBB3550/5FB5E480" Ref="#PWR?"  Part="1"
+AR Path="/5FBB3550/5FB5E480" Ref="#PWR033"  Part="1"
 AR Path="/5FB5E480" Ref="#PWR?"  Part="1"
 AR Path="/5F78DB3E/5FB5E480" Ref="#PWR?"  Part="1"
-F 0 "#PWR?" H 3650 3600 50  0001 C CNN
+F 0 "#PWR033" H 3650 3600 50  0001 C CNN
 F 1 "GND" H 3655 3677 50  0000 C CNN
 F 2 "" H 3650 3850 50  0001 C CNN
@@
 $EndComp
 $Comp
-L power:GND #PWR?
+L power:GND #PWR034
 U 1 1 5FB5E486
 P 3800 3850
-AR Path="/5FBB3550/5FB5E486" Ref="#PWR?"  Part="1"
+AR Path="/5FBB3550/5FB5E486" Ref="#PWR034"  Part="1"
 AR Path="/5FB5E486" Ref="#PWR?"  Part="1"
 AR Path="/5F78DB3E/5FB5E486" Ref="#PWR?"  Part="1"
-F 0 "#PWR?" H 3800 3600 50  0001 C CNN
+F 0 "#PWR034" H 3800 3600 50  0001 C CNN
 F 1 "GND" H 3805 3677 50  0000 C CNN
 F 2 "" H 3800 3850 50  0001 C CNN
@@
 $EndComp
 $Comp
-L power:GND #PWR?
+L power:GND #PWR035
 U 1 1 5FB5E48C
 P 3950 3850
-AR Path="/5FBB3550/5FB5E48C" Ref="#PWR?"  Part="1"
+AR Path="/5FBB3550/5FB5E48C" Ref="#PWR035"  Part="1"
 AR Path="/5FB5E48C" Ref="#PWR?"  Part="1"
 AR Path="/5F78DB3E/5FB5E48C" Ref="#PWR?"  Part="1"
-F 0 "#PWR?" H 3950 3600 50  0001 C CNN
+F 0 "#PWR035" H 3950 3600 50  0001 C CNN
 F 1 "GND" H 3955 3677 50  0000 C CNN
 F 2 "" H 3950 3850 50  0001 C CNN
@@
 	3800 3100 3600 3100
 $Comp
-L power:GND #PWR?
+L power:GND #PWR031
 U 1 1 5FB5E49D
 P 3200 3500
-AR Path="/5FBB3550/5FB5E49D" Ref="#PWR?"  Part="1"
+AR Path="/5FBB3550/5FB5E49D" Ref="#PWR031"  Part="1"
 AR Path="/5FB5E49D" Ref="#PWR?"  Part="1"
 AR Path="/5F78DB3E/5FB5E49D" Ref="#PWR?"  Part="1"
-F 0 "#PWR?" H 3200 3250 50  0001 C CNN
+F 0 "#PWR031" H 3200 3250 50  0001 C CNN
 F 1 "GND" H 3050 3450 50  0000 C CNN
 F 2 "" H 3200 3500 50  0001 C CNN
@@
 $EndComp
 NoConn ~ 3600 3300
-$Comp
-L power:+5V #PWR?
-U 1 1 5FB5E4A6
-P 3950 2750
-AR Path="/5FB5E4A6" Ref="#PWR?"  Part="1"
-AR Path="/5F78DB3E/5FB5E4A6" Ref="#PWR?"  Part="1"
-AR Path="/5FBB3550/5FB5E4A6" Ref="#PWR?"  Part="1"
-F 0 "#PWR?" H 3950 2600 50  0001 C CNN
-F 1 "+5V" H 3965 2923 50  0000 C CNN
-F 2 "" H 3950 2750 50  0001 C CNN
-F 3 "" H 3950 2750 50  0001 C CNN
-	1    3950 2750
-	1    0    0    -1
-$EndComp
 Wire Wire Line
 	3950 2750 3950 2900
@@
 Wire Wire Line
 	3650 3200 5000 3200
+Text HLabel 3950 2750 1    50   Input ~ 0
+V_OUT
 $EndSCHEMATC

Commit message: repair footprint of P and N MOS, add order codes for JLCPCB, preparing for fab
Parts:
- C22, C23, D7, D8, D9, J1, R10, R6, R7, R8, R9: JLCPCB_CORRECTION (none) -> 0;0;0
- D10, D11: JLCPCB_CORRECTION 0;0;180 -> 0;0;0
- Q1, Q2: JLCPCB_CORRECTION (none) -> 0;0;180; LCSC (none) -> C20526
Changed lines of the file:
@@
 F 3 "~" H 4500 2500 50  0001 C CNN
 F 4 "C4109" H 4500 2500 50  0001 C CNN "LCSC"
+F 5 "0;0;0" H 4500 2500 50  0001 C CNN "JLCPCB_CORRECTION"
 	1    4500 2500
 	1    0    0    -1
@@
 F 3 "~" H 6500 3100 50  0001 C CNN
 F 4 "C25744" H 6500 3100 50  0001 C CNN "LCSC"
+F 5 "0;0;0" H 6500 3100 50  0001 C CNN "JLCPCB_CORRECTION"
 	1    6500 3100
 	0    1    1    0
@@
 F 3 "~" H 7550 2700 50  0001 C CNN
 F 4 "C25744" H 7550 2700 50  0001 C CNN "LCSC"
+F 5 "0;0;0" H 7550 2700 50  0001 C CNN "JLCPCB_CORRECTION"
 	1    7550 2700
 	0    1    1    0
@@
 F 3 "~" H 5900 2250 50  0001 C CNN
 F 4 "C1525" H 5900 2250 50  0001 C CNN "LCSC"
+F 5 "0;0;0" H 5900 2250 50  0001 C CNN "JLCPCB_CORRECTION"
 	1    5900 2250
 	0    1    1    0
@@
 F 3 "~" H 6550 2350 50  0001 C CNN
 F 4 "C25792" H 6550 2350 50  0001 C CNN "LCSC"
+F 5 "0;0;0" H 6550 2350 50  0001 C CNN "JLCPCB_CORRECTION"
 	1    6550 2350
 	1    0    0    -1
@@
 F 3 "~" H 6850 2350 50  0001 C CNN
 F 4 "C25792" H 6850 2350 50  0001 C CNN "LCSC"
+F 5 "0;0;0" H 6850 2350 50  0001 C CNN "JLCPCB_CORRECTION"
 	1    6850 2350
 	1    0    0    -1
@@
 F 3 "~" H 6550 1950 50  0001 C CNN
 F 4 "C72043" H 6550 1950 50  0001 C CNN "LCSC"
-F 5 "0;0;180" H 6550 1950 50  0001 C CNN "JLCPCB_CORRECTION"
+F 5 "0;0;0" H 6550 1950 50  0001 C CNN "JLCPCB_CORRECTION"
 	1    6550 1950
 	0    -1   -1   0
@@
 F 3 "~" H 6850 1950 50  0001 C CNN
 F 4 "C72043" H 6850 1950 50  0001 C CNN "LCSC"
-F 5 "0;0;180" H 6850 1950 50  0001 C CNN "JLCPCB_CORRECTION"
+F 5 "0;0;0" H 6850 1950 50  0001 C CNN "JLCPCB_CORRECTION"
 	1    6850 1950
 	0    -1   -1   0
@@
 F 2 "Package_TO_SOT_SMD:SOT-23" H 8250 2800 50  0001 C CNN
 F 3 "~" H 8050 2700 50  0001 C CNN
+F 4 " C20526" H 8050 2700 50  0001 C CNN "LCSC"
+F 5 "0;0;180" H 8050 2700 50  0001 C CNN "JLCPCB_CORRECTION"
 	1    8050 2700
 	1    0    0    -1
@@
 F 2 "Package_TO_SOT_SMD:SOT-23" H 7450 3200 50  0001 C CNN
 F 3 "~" H 7250 3100 50  0001 C CNN
+F 4 " C20526" H 7250 3100 50  0001 C CNN "LCSC"
+F 5 "0;0;180" H 7250 3100 50  0001 C CNN "JLCPCB_CORRECTION"
 	1    7250 3100
 	1    0    0    1
@@
 F 3 "~" H 5900 1950 50  0001 C CNN
 F 4 "C23733" H 5900 1950 50  0001 C CNN "LCSC"
+F 5 "0;0;0" H 5900 1950 50  0001 C CNN "JLCPCB_CORRECTION"
 	1    5900 1950
 	0    1    1    0
@@
 F 3 "~" H 3450 3050 50  0001 C CNN
 F 4 "ručně" H 3300 3100 50  0001 C CNN "LCSC"
+F 5 "0;0;0" H 3300 3100 50  0001 C CNN "JLCPCB_CORRECTION"
 	1    3300 3100
 	1    0    0    -1
@@
 F 3 "https://www.littelfuse.com/~/media/electronics/datasheets/tvs_diode_arrays/littelfuse_tvs_diode_array_sd_c_datasheet.pdf.pdf" H 3650 3600 50  0001 C CNN
 F 4 "neosazovat" H 3650 3600 50  0001 C CNN "LCSC"
+F 5 "0;0;0" H 3650 3600 50  0001 C CNN "JLCPCB_CORRECTION"
 	1    3650 3600
 	0    -1   -1   0
@@
 F 3 "https://www.littelfuse.com/~/media/electronics/datasheets/tvs_diode_arrays/littelfuse_tvs_diode_array_sd_c_datasheet.pdf.pdf" H 3800 3600 50  0001 C CNN
 F 4 "neosazovat" H 3800 3600 50  0001 C CNN "LCSC"
+F 5 "0;0;0" H 3800 3600 50  0001 C CNN "JLCPCB_CORRECTION"
 	1    3800 3600
 	0    -1   -1   0
@@
 F 3 "https://www.littelfuse.com/~/media/electronics/datasheets/tvs_diode_arrays/littelfuse_tvs_diode_array_sd_c_datasheet.pdf.pdf" H 3950 3600 50  0001 C CNN
 F 4 "neosazovat" H 3950 3600 50  0001 C CNN "LCSC"
+F 5 "0;0;0" H 3950 3600 50  0001 C CNN "JLCPCB_CORRECTION"
 	1    3950 3600
 	0    -1   -1   0
